File: pcb/led_controller.kicad_pcb (KiCad board)
At the start: 2 copper layers, 75 parts, among them IC1 ATTINY2313A-S, P1 POSITIVE_OUT_1, P10 NEGATIVE_OUT_1, P11 NEGATIVE_OUT_2, P12 NEGATIVE_OUT_2, P13 NEGATIVE_OUT_2, P14 ISP, P15 +12v IN, P16 GND IN, P2 POSITIVE_OUT_2, P3 POSITIVE_OUT_3, P4 POSITIVE_OUT_4, P5 ESP8266, P6 POSITIVE_OUT_5, P7 POSITIVE_OUT_6, P8 NEGATIVE_OUT_1, P9 NEGATIVE_OUT_1, Q1 MOSFET_P, Q10 MOSFET_N, Q2 MOSFET_P, Q3 MOSFET_P, Q4 MOSFET_P, Q5 MOSFET_P, Q6 MOSFET_P, Q7 BS170, Q8 BS170, Q9 MOSFET_N, SW1 B1, SW2 B2, U1 TC4426A, U2 TC4426A, U3 TC4426A, U4 TC4427A, U5 MCP1700, U6 MC34063, X1 20MHz

Commit message: some 3D models
Parts:
- moved 1pin 5.72 mm to (177.2, 131.1)
- moved 1pin 5.72 mm to (108.0, 131.1)

Commit message: second PCB
Parts:
- added 1pin: VAL**, Connect:1pin, F.Cu at (108.0, 56.2)
- added 1pin: VAL**, Connect:1pin, F.Cu at (129.9, 28.6)
- added 1pin: VAL**, Connect:1pin, F.Cu at (134.9, 28.6)
- added 1pin: VAL**, Connect:1pin, F.Cu at (140.0, 28.6)
- added 1pin: VAL**, Connect:1pin, F.Cu at (145.1, 28.6)
- added 1pin: VAL**, Connect:1pin, F.Cu at (150.2, 28.6)
- added 1pin: VAL**, Connect:1pin, F.Cu at (155.3, 28.6)
- added 1pin: VAL**, Connect:1pin, F.Cu at (160.3, 28.6)
- added 1pin: VAL**, Connect:1pin, F.Cu at (165.4, 28.6)
- added 1pin: VAL**, Connect:1pin, F.Cu at (170.5, 28.6)
- added 1pin: VAL**, Connect:1pin, F.Cu at (177.2, 94.9)
- added 1pin: VAL**, Connect:1pin, F.Cu at (177.2, 56.2)
- added 1pin: VAL**, Connect:1pin, F.Cu at (108.0, 94.9)
- added 1pin: VAL**, Connect:1pin, F.Cu at (108.0, 28.6)
- added 1pin: VAL**, Connect:1pin, F.Cu at (177.2, 28.6)
- added 1pin: VAL**, Connect:1pin, F.Cu at (114.6, 28.6)
- added 1pin: VAL**, Connect:1pin, F.Cu at (119.7, 28.6)
- added 1pin: VAL**, Connect:1pin, F.Cu at (124.8, 28.6)
- added P17: GND_IN, connectors:1PIN_DG306, F.Cu at (177.2, 45.1)
- added P18: GND_OUT, connectors:1PIN_DG306, F.Cu at (129.9, 36.2)
- added P19: VDD_IN, connectors:1PIN_DG306, F.Cu at (177.2, 50.2)
- added P20: VDD_OUT, connectors:1PIN_DG306, F.Cu at (124.8, 36.2)
- added P21: GND_OUT, connectors:1PIN_DG306, F.Cu at (119.7, 36.2)
- added P22: VDD_OUT, connectors:1PIN_DG306, F.Cu at (165.4, 36.2)
- added P23: GND_OUT, connectors:1PIN_DG306, F.Cu at (140.0, 36.2)
- added P24: VDD_OUT, connectors:1PIN_DG306, F.Cu at (134.9, 36.2)
- added P25: GND_OUT, connectors:1PIN_DG306, F.Cu at (150.2, 36.2)
- added P26: VDD_OUT, connectors:1PIN_DG306, F.Cu at (145.1, 36.2)
- added P27: GND_OUT, connectors:1PIN_DG306, F.Cu at (160.3, 36.2)
- added P28: VDD_OUT, connectors:1PIN_DG306, F.Cu at (155.3, 36.2)
- added P29: GND_OUT, connectors:1PIN_DG306, F.Cu at (170.5, 36.2)
- added P30: VDD_OUT, connectors:1PIN_DG306, F.Cu at (114.6, 36.2)
- P15: value +12v IN -> +12v_IN
- P16: value GND IN -> GND_IN
- moved C11 4.13 mm to (176.5, 105.4), turned to 270 degrees
Routing:
- net Net-(P19-Pad1): track 0.00 -> 145.2 mm
- added copper zone on B.Cu, net /Power Supply/GND2
