File: led_controller_pcb/led_controller_pcb.kicad_pcb (KiCad board)
At the start: 2 copper layers, 34.9 x 57.8 mm, 94 parts, among them J1 DCDC, J10 PASSIVE_OUT, J11 VPP, J12 OUT, J13 VPP, J14 OUT, J15 VPP, J16 PASSIVE_OUT, J17 VPP, J18 OUT, J19 VPP, J2 DEBUG, J20 OUT, J21 LINE1_IN, J22 LINE2_IN, J24 HV_LINE, J25 HV_OUT, J26 HV_LINE, J27 HV_OUT, J28 PSU_LINE1, J29 PSU_LINE2, J3 VPP, J31 PSU_GND, J32 PSU_VOUT, J4 PASSIVE_OUT, J5 VPP, J6 OUT, J7 VPP, J8 OUT, J9 VPP, Q1 IRF540N, Q10 BT136-600, Q2 IRF540N, Q3 IRF540N, Q4 IRF540N, Q5 IRF540N, Q6 IRF540N, Q7 BC549, Q8 BC549, Q9 BT136-600, SW1 BUTTON, SW2 BUTTON, U1 ESP-12E, U2 TC4427A, U3 TC4427A, U4 TC4427A, U5 STM32F030F4Px, U6 MOC3023M, U7 MOC3023M, U8 H11AA1, Y1 8MHz

Commit message: pcb all connected
Parts:
- removed D1: LED, LED_THT:LED_D5.0mm
- removed R5: 4.7k, Resistor_SMD:R_0805_2012Metric
- C1, C2, C5, C7, R10, R11, R12, R15, R4, R6: moved to B.Cu
- R9: moved to F.Cu
- moved C1 142.9 mm to (72.4, 67.0)
- moved R10 129.4 mm to (61.0, 30.5), turned to 180 degrees
- moved R28 93.9 mm to (67.6, 54.6)
- moved R6 88.0 mm to (73.4, 53.7)
- moved R11 87.1 mm to (80.0, 32.4)
- moved R16 86.0 mm to (78.4, 30.2), turned to -90 degrees
- moved C2 80.1 mm to (71.5, 30.8), turned to 180 degrees
- moved R4 73.0 mm to (60.9, 32.7)
- moved C5 72.8 mm to (70.8, 18.7), turned to 90 degrees
- moved R12 72.3 mm to (66.7, 26.0), turned to 90 degrees
- moved D2 63.4 mm to (75.2, 56.8), turned to 180 degrees
- moved R13 62.1 mm to (80.0, 42.5)
- moved C7 56.3 mm to (64.9, 5.00), turned to -90 degrees
- moved R8 45.8 mm to (82.2, 12.4), turned to -90 degrees
- moved R7 37.9 mm to (80.0, 15.7)
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Connections:
- R6 pad 1: Net-(R6-Pad1) -> Net-(D2-Pad2)
- R6 pad 2: Net-(D2-Pad2) -> Net-(R6-Pad2)
- U1 pad 12: Net-(R6-Pad1) -> Net-(U1-Pad12)
- U1 pad 6: Net-(U1-Pad6) -> Net-(R6-Pad2)
- U3 pad 2: /TIM15_CH2 -> /TIM3_CH2
- U3 pad 4: /TIM3_CH2 -> /TIM15_CH2
Routing:
- net GND: track 178.9 -> 365.5 mm, vias 0 -> 7
- net /GPO2: track 0.00 -> 62.2 mm, vias 0 -> 4
- net /GPO1: track 0.00 -> 58.2 mm, vias 0 -> 4
- net /AC_SYNC: track 0.00 -> 43.3 mm, vias 0 -> 1
- net Net-(R6-Pad2): track 0.00 -> 26.1 mm, vias 0 -> 3
- net /TIM3_CH2: track 0.70 -> 19.8 mm, vias 0 -> 2
- net +3V3: track 122.3 -> 139.4 mm, vias 1 -> 2
- net Net-(R10-Pad2): track 9.30 -> 25.9 mm, vias 0 -> 1
- net Net-(Q5-Pad1): track 0.00 -> 10.8 mm
- net Net-(R4-Pad1): track 0.00 -> 9.64 mm, vias 0 -> 1
- net Net-(Q6-Pad1): track 0.00 -> 4.40 mm
- net VDD: track 216.8 -> 220.9 mm
- net Net-(C4-Pad1): track 6.53 -> 10.6 mm
- net /TIM3_CH1: track 24.4 -> 28.2 mm
- net /TIM15_CH2: track 14.7 -> 11.1 mm
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Other:
- board size 34.9 x 57.8 mm -> 50.2 x 99.7 mm

Commit message: finish pcb
Parts:
- added C9: 100n, Capacitor_SMD:C_0805_2012Metric, B.Cu at (141.6, 58.1)
- moved J15 86.0 mm to (162.6, 134.0)
- moved J7 86.0 mm to (162.6, 144.1)
- moved REF** 86.0 mm to (154.3, 140.3)
- moved U1 86.0 mm to (130.2, 81.9)
- moved C1 86.0 mm to (140.3, 119.7)
- moved C2 86.0 mm to (139.4, 83.5)
- moved C3 86.0 mm to (139.7, 59.3)
- moved C4 86.0 mm to (144.9, 71.8)
- moved C5 86.0 mm to (138.8, 71.4)
- moved C6 86.0 mm to (145.7, 75.1)
- moved C7 86.0 mm to (132.8, 57.7)
- moved C8 86.0 mm to (130.8, 55.9)
- moved D4 86.0 mm to (120.0, 106.7)
- moved D5 86.0 mm to (124.5, 106.7)
- moved J1 86.0 mm to (138.0, 64.4)
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Connections:
- U8 pad 1: Net-(D4-Pad1) -> Net-(D5-Pad1)
- U8 pad 2: Net-(D5-Pad1) -> Net-(D4-Pad1)
Routing:
- net GND: track 365.5 -> 368.4 mm
- net +3V3: track 139.4 -> 141.4 mm
- net Net-(D5-Pad1): track 10.7 -> 8.70 mm
Other:
- net class Default: trace_width 0.25 -> 0.3
- rule solder_mask_min_width: 0.25 -> 0.3
