File: led_controller_pcb/led_controller_pcb.sch (KiCad schematic (older format))
At the start: 91 parts, among them J1 DCDC, J10 PASSIVE_OUT, J11 VPP, J12 OUT, J13 VPP, J14 OUT, J15 VPP, J16 PASSIVE_OUT, J17 VPP, J18 OUT, J19 VPP, J2 DEBUG, J20 OUT, J21 LINE1_IN, J22 LINE2_IN, J24 HV_LINE, J25 HV_OUT, J26 HV_LINE, J27 HV_OUT, J28 PSU_LINE1, J29 PSU_LINE2, J3 VPP, J31 PSU_GND, J32 PSU_VOUT, J4 PASSIVE_OUT, J5 VPP, J6 OUT, J7 VPP, J8 OUT, J9 VPP, Q1 IRF540N, Q10 BT136-600, Q2 IRF540N, Q3 IRF540N, Q4 IRF540N, Q5 IRF540N, Q6 IRF540N, Q7 BC549, Q8 BC549, Q9 BT136-600, SW1 BUTTON, SW2 BUTTON, U1 ESP-12E, U2 TC4427A, U3 TC4427A, U4 TC4427A, U5 STM32F030F4Px, U6 MOC3023M, U7 MOC3023M, U8 H11AA1, Y1 8MHz

Commit message: add resistor
Parts:
- gave numbers to parts that had none: 1
Changed lines of the file:
@@
 	2700 9400 2350 9400
 $Comp
-L Device:R R?
+L Device:R R5
 U 1 1 5D9DC575
 P 4550 8400
-F 0 "R?" V 4450 8400 50  0000 C CNN
+F 0 "R5" V 4450 8400 50  0000 C CNN
 F 1 "4.7k" V 4550 8400 50  0000 C CNN
 F 2 "Resistor_SMD:R_0805_2012Metric" V 4480 8400 50  0001 C CNN
@@
 $EndComp
 $Comp
-L power:+3.3V #PWR?
+L power:+3.3V #PWR0117
 U 1 1 5D9DED9E
 P 4550 8100
-F 0 "#PWR?" H 4550 7950 50  0001 C CNN
+F 0 "#PWR0117" H 4550 7950 50  0001 C CNN
 F 1 "+3.3V" H 4565 8273 50  0000 C CNN
 F 2 "" H 4550 8100 50  0001 C CNN

Commit message: update schematic
Parts:
- U6, U7: symbol led_controller_pcb-rescue:MOC3023M-Relay_SolidState -> led_controller_pcb-rescue:MOC3023M-Relay_SolidState-led_controller_pcb-rescue
Changed lines of the file:
@@
 	14000 2150 13550 2150
 $Comp
-L led_controller_pcb-rescue:MOC3023M-Relay_SolidState U6
+L led_controller_pcb-rescue:MOC3023M-Relay_SolidState-led_controller_pcb-rescue U6
 U 1 1 5D957503
 P 13250 2050
@@
 	14150 4400 14400 4400
 $Comp
-L led_controller_pcb-rescue:MOC3023M-Relay_SolidState U7
+L led_controller_pcb-rescue:MOC3023M-Relay_SolidState-led_controller_pcb-rescue U7
 U 1 1 5DA06959
 P 13250 4100

Commit message: wip on adding a separate connector for high voltage
Parts:
- added C11, C13, C14, C15: 100n, Capacitor_SMD:C_0805_2012Metric, symbol Device:C
- added C12: 470uF, Capacitor_THT:CP_Radial_D8.0mm_P3.50mm, symbol Device:CP
- added J23: PSU_VOUT_LOW, connectors:1PIN_DG306, symbol Connector:Screw_Terminal_01x01
- C8: value 470uF -> 220uF; footprint Capacitor_THT:CP_Radial_D8.0mm_P3.50mm -> Capacitor_SMD:CP_Elec_6.3x7.7
Connections:
- net GND: now also C11.2, C12.2, C13.2, C14.2, C15.2
- net VDD: now also C13.1, C14.1, C15.1, J23.1 (Pin_1); no longer J11.1 (Pin_1), J13.1 (Pin_1), J15.1 (Pin_1), J17.1 (Pin_1), J19.1 (Pin_1), J3.1 (Pin_1), J32.1 (Pin_1), J5.1 (Pin_1), J7.1 (Pin_1), J9.1 (Pin_1)
- new net VPP: C11.1, C12.1, J11.1 (Pin_1), J13.1 (Pin_1), J15.1 (Pin_1), J17.1 (Pin_1), J19.1 (Pin_1), J3.1 (Pin_1), J32.1 (Pin_1), J5.1 (Pin_1), J7.1 (Pin_1), J9.1 (Pin_1)
Other:
- moved on the sheet: C7, C8

Commit message: cosmetic fixes
Parts:
- removed C8: 220uF, Capacitor_SMD:CP_Elec_6.3x7.7, symbol Device:CP
- added C16: 220uF, Capacitor_SMD:CP_Elec_6.3x7.7, symbol Device:CP
- C3: footprint Capacitor_THT:CP_Radial_D8.0mm_P3.50mm -> Capacitor_SMD:CP_Elec_6.3x7.7
- J21: value LINE1_IN -> HV_IN_LIVE
- J22: value LINE2_IN -> HV_IN_NEUT
- J28: value PSU_LINE1 -> PSU_LIVE
- J29: value PSU_LINE2 -> PSU_NEUT
Connections:
- net GND: now also C16.2
- net VDD: now also C16.1
- net LINE1 renamed LIVE
- net LINE2 renamed NEUT
Changed lines of the file:
@@
 Comment9 ""
 $EndDescr
+Connection ~ 4550 9000
+Connection ~ 14200 8900
+Connection ~ 2350 9400
+Connection ~ 14150 3850
+Connection ~ 15550 5700
+Connection ~ 4150 6250
+Connection ~ 2700 9000
+Connection ~ 14200 8400
+Connection ~ 5150 10300
+Connection ~ 9300 8550
+Connection ~ 6350 6250
+Connection ~ 8550 8800
+Connection ~ 14150 1800
+Connection ~ 2700 9400
+Connection ~ 7650 10000
+Connection ~ 14500 6100
+Connection ~ 8150 10000
+Connection ~ 1800 4150
+Connection ~ 14500 5300
+Connection ~ 14200 8650
 Connection ~ 6350 4500
-Connection ~ 15550 5700
-Connection ~ 2350 9400
 Connection ~ 8600 6250
-Connection ~ 4550 9000
-Connection ~ 9300 8550
+Connection ~ 8600 4500
+Connection ~ 4150 4500
+Connection ~ 5500 10100
 Connection ~ 1850 3850
-Connection ~ 14200 8400
+Connection ~ 3150 9000
+Connection ~ 8550 9000
+Connection ~ 12400 2850
 Connection ~ 12400 4900
-Connection ~ 7650 10000
-Connection ~ 6350 6250
-Connection ~ 14200 8900
-Connection ~ 14150 1800
-Connection ~ 4150 4500
-Connection ~ 14150 3850
-Connection ~ 8600 4500
-Connection ~ 8150 10000
-Connection ~ 2700 9000
-Connection ~ 5150 10300
-Connection ~ 3150 9000
-Connection ~ 14500 5300
-Connection ~ 12400 2850
-Connection ~ 5500 10100
-Connection ~ 2700 9400
-Connection ~ 8550 8800
-Connection ~ 14200 8650
-Connection ~ 1800 4150
-Connection ~ 4150 6250
-Connection ~ 14500 6100
-Connection ~ 8550 9000
-NoConn ~ 3250 10000
-NoConn ~ 3250 9600
 NoConn ~ 4450 9500
-NoConn ~ 15500 5600
 NoConn ~ 3250 10100
 NoConn ~ 4450 9400
-NoConn ~ 3250 9700
+NoConn ~ 3250 10000
 NoConn ~ 3250 9900
 NoConn ~ 4450 9200
+NoConn ~ 3250 9600
+NoConn ~ 15500 5600
 NoConn ~ 3250 9800
+NoConn ~ 3250 9700
 Wire Wire Line
 	1550 4850 1550 4750
@@
 	11200 10650 11200 10550
 Wire Wire Line
+	11725 9200 11725 9300
+Wire Wire Line
+	11725 9700 11725 9600
+Wire Wire Line
 	12000 2850 11750 2850
 Wire Wire Line
 	12000 4900 11750 4900
-Wire Wire Line
-	12150 9200 12150 9300
-Wire Wire Line
-	12150 9700 12150 9600
 Wire Wire Line
 	12300 2850 12400 2850
@@
 GPO2
 Text Label 12750 7650 0    50   ~ 0
-LINE1
+LIVE
 Text Label 12750 7900 0    50   ~ 0
-LINE2
+NEUT
 Text Label 13750 5300 0    50   ~ 0
-LINE2
+NEUT
 Text Label 13750 6100 0    50   ~ 0
-LINE1
+LIVE
 Text Label 14150 7650 2    50   ~ 0
-LINE1
+LIVE
 Text Label 14150 7900 2    50   ~ 0
-LINE2
+NEUT
 Text Label 14400 1050 0    50   ~ 0
-LINE1
+LIVE
 Text Label 14400 2350 0    50   ~ 0
-LINE2
+NEUT
 Text Label 14400 3100 0    50   ~ 0
-LINE1
+LIVE
 Text Label 14400 4400 0    50   ~ 0
-LINE2
+NEUT
 Text Label 15700 5700 0    50   ~ 0
 AC_SYNC
@@
 $EndComp
 $Comp
-L power:VDD #PWR0111
-U 1 1 5D86887E
-P 12150 9200
-F 0 "#PWR0111" H 12150 9050 50  0001 C CNN
-F 1 "VDD" H 12150 9400 50  0000 C CNN
-F 2 "" H 12150 9200 50  0001 C CNN
-F 3 "" H 12150 9200 50  0001 C CNN
-	1    12150 9200
+L power:VDD #PWR075
+U 1 1 00000000
+P 11725 9200
+F 0 "#PWR075" H 11725 9050 50  0001 C CNN
+F 1 "VDD" H 11725 9400 50  0000 C CNN
+F 2 "" H 11725 9200 50  0001 C CNN
+F 3 "" H 11725 9200 50  0001 C CNN
+	1    11725 9200
 	1    0    0    -1
 $EndComp
@@
 $EndComp
 $Comp
-L power:GND #PWR065
-U 1 1 5D85D891
-P 12150 9700
-F 0 "#PWR065" H 12150 9450 50  0001 C CNN
-F 1 "GND" H 12154 9545 50  0001 C CNN
-F 2 "" H 12150 9700 50  0001 C CNN
-F 3 "" H 12150 9700 50  0001 C CNN
-	1    12150 9700
+L power:GND #PWR076
+U 1 1 00000000
+P 11725 9700
+F 0 "#PWR076" H 11725 9450 50  0001 C CNN
+F 1 "GND" H 11729 9545 50  0001 C CNN
+F 2 "" H 11725 9700 50  0001 C CNN
+F 3 "" H 11725 9700 50  0001 C CNN
+	1    11725 9700
 	1    0    0    -1
 $EndComp
@@
 P 12450 7650
 F 0 "J21" H 12500 7550 50  0000 C CNN
-F 1 "LINE1_IN" H 12700 7650 50  0000 C CNN
+F 1 "HV_IN_LIVE" H 12750 7650 50  0000 C CNN
 F 2 "connectors:1PIN_DG306" H 12450 7650 50  0001 C CNN
 F 3 "~" H 12450 7650 50  0001 C CNN
@@
 P 12450 7900
 F 0 "J22" H 12500 7800 50  0000 C CNN
-F 1 "LINE2_IN" H 12700 7900 50  0000 C CNN
+F 1 "HV_IN_NEUT" H 12775 7900 50  0000 C CNN
 F 2 "connectors:1PIN_DG306" H 12450 7900 50  0001 C CNN
 F 3 "~" H 12450 7900 50  0001 C CNN
@@
 P 14450 7650
 F 0 "J28" H 14550 7550 50  0000 C CNN
-F 1 "PSU_LINE1" H 14750 7650 50  0000 C CNN
+F 1 "PSU_LIVE" H 14750 7650 50  0000 C CNN
 F 2 "connectors:1PIN_DG306" H 14450 7650 50  0001 C CNN
 F 3 "~" H 14450 7650 50  0001 C CNN
@@
 P 14450 7900
 F 0 "J29" H 14550 7800 50  0000 C CNN
-F 1 "PSU_LINE2" H 14750 7900 50  0000 C CNN
+F 1 "PSU_NEUT" H 14750 7900 50  0000 C CNN
 F 2 "connectors:1PIN_DG306" H 14450 7900 50  0001 C CNN
 F 3 "~" H 14450 7900 50  0001 C CNN
@@
 P 14450 8400
 F 0 "J31" H 14550 8300 50  0000 C CNN
-F 1 "PSU_GND" H 14750 8400 50  0000 C CNN
+F 1 "PSU_GND" H 14725 8400 50  0000 C CNN
 F 2 "connectors:1PIN_DG306" H 14450 8400 50  0001 C CNN
 F 3 "~" H 14450 8400 50  0001 C CNN
@@
 P 14450 8900
 F 0 "J23" H 14550 8800 50  0000 C CNN
-F 1 "PSU_VOUT_LOW" H 14850 8900 50  0000 C CNN
+F 1 "PSU_VOUT_LOW" H 14850 8925 50  0000 C CNN
 F 2 "connectors:1PIN_DG306" H 14450 8900 50  0001 C CNN
 F 3 "~" H 14450 8900 50  0001 C CNN
@@
 F 0 "C3" H 2168 5046 50  0000 L CNN
 F 1 "470uF" H 2168 4955 50  0000 L CNN
-F 2 "Capacitor_THT:CP_Radial_D8.0mm_P3.50mm" H 2088 4850 50  0001 C CNN
+F 2 "Capacitor_SMD:CP_Elec_6.3x7.7" H 2088 4850 50  0001 C CNN
 F 3 "~" H 2050 5000 50  0001 C CNN
 	1    2050 5000
@@
 $EndComp
 $Comp
-L Device:CP C8
-U 1 1 5D85D8B7
-P 12150 9450
-F 0 "C8" H 12268 9496 50  0000 L CNN
-F 1 "220uF" H 12268 9405 50  0000 L CNN
-F 2 "Capacitor_SMD:CP_Elec_6.3x7.7" H 12188 9300 50  0001 C CNN
-F 3 "~" H 12150 9450 50  0001 C CNN
-	1    12150 9450
-	1    0    0    -1
-$EndComp
+L Device:CP C16
+U 1 1 00000000
+P 11725 9450
+F 0 "C16" H 11843 9496 50  0000 L CNN
+F 1 "220uF" H 11843 9405 50  0000 L CNN
+F 2 "Capacitor_SMD:CP_Elec_6.3x7.7" H 11763 9300 50  0001 C CNN
+F 3 "~" H 11725 9450 50  0001 C CNN
+	1    11725 9450
+	1    0    0    -1
+$EndComp

Commit message: update 0805 components to have larger pads
Parts:
- C1, C10, C11, C13, C14, C15, C2, C4, C5, C6, C7, C9: footprint Capacitor_SMD:C_0805_2012Metric -> Capacitor_SMD:C_0805_2012Metric_Pad1.15x1.40mm_HandSolder
- R10, R11, R12, R13, R14, R15, R16, R18, R19, R2, R20, R21, R22, R23, R28, R3, R4, R5, R6, R7, R8, R9: footprint Resistor_SMD:R_0805_2012Metric -> Resistor_SMD:R_0805_2012Metric_Pad1.15x1.40mm_HandSolder
Changed lines of the file:
@@
 F 0 "R2" H 2281 9646 50  0000 R CNN
 F 1 "150k" H 2281 9555 50  0000 R CNN
-F 2 "Resistor_SMD:R_0805_2012Metric" V 2280 9600 50  0001 C CNN
+F 2 "Resistor_SMD:R_0805_2012Metric_Pad1.15x1.40mm_HandSolder" V 2280 9600 50  0001 C CNN
 F 3 "~" H 2350 9600 50  0001 C CNN
 	1    2350 9600
@@
 F 0 "R3" V 2800 9000 50  0000 C CNN
 F 1 "4.7k" V 2900 9000 50  0000 C CNN
-F 2 "Resistor_SMD:R_0805_2012Metric" V 2830 9000 50  0001 C CNN
+F 2 "Resistor_SMD:R_0805_2012Metric_Pad1.15x1.40mm_HandSolder" V 2830 9000 50  0001 C CNN
 F 3 "~" H 2900 9000 50  0001 C CNN
 	1    2900 9000
@@
 F 0 "R4" V 2800 9200 50  0000 C CNN
 F 1 "4.7k" V 2900 9200 50  0000 C CNN
-F 2 "Resistor_SMD:R_0805_2012Metric" V 2830 9200 50  0001 C CNN
+F 2 "Resistor_SMD:R_0805_2012Metric_Pad1.15x1.40mm_HandSolder" V 2830 9200 50  0001 C CNN
 F 3 "~" H 2900 9200 50  0001 C CNN
 	1    2900 9200
@@
 F 0 "R7" H 4220 4746 50  0000 L CNN
 F 1 "47k" H 4220 4655 50  0000 L CNN
-F 2 "Resistor_SMD:R_0805_2012Metric" V 4080 4700 50  0001 C CNN
+F 2 "Resistor_SMD:R_0805_2012Metric_Pad1.15x1.40mm_HandSolder" V 4080 4700 50  0001 C CNN
 F 3 "~" H 4150 4700 50  0001 C CNN
 	1    4150 4700
@@
 F 0 "R8" H 4220 6496 50  0000 L CNN
 F 1 "47k" H 4220 6405 50  0000 L CNN
-F 2 "Resistor_SMD:R_0805_2012Metric" V 4080 6450 50  0001 C CNN
+F 2 "Resistor_SMD:R_0805_2012Metric_Pad1.15x1.40mm_HandSolder" V 4080 6450 50  0001 C CNN
 F 3 "~" H 4150 6450 50  0001 C CNN
 	1    4150 6450
@@
 F 0 "R5" V 4450 8400 50  0000 C CNN
 F 1 "4.7k" V 4550 8400 50  0000 C CNN
-F 2 "Resistor_SMD:R_0805_2012Metric" V 4480 8400 50  0001 C CNN
+F 2 "Resistor_SMD:R_0805_2012Metric_Pad1.15x1.40mm_HandSolder" V 4480 8400 50  0001 C CNN
 F 3 "~" H 4550 8400 50  0001 C CNN
 	1    4550 8400
@@
 F 0 "R6" V 4550 10250 50  0000 C CNN
 F 1 "4.7k" V 4600 10450 50  0000 C CNN
-F 2 "Resistor_SMD:R_0805_2012Metric" V 4530 10450 50  0001 C CNN
+F 2 "Resistor_SMD:R_0805_2012Metric_Pad1.15x1.40mm_HandSolder" V 4530 10450 50  0001 C CNN
 F 3 "~" H 4600 10450 50  0001 C CNN
 	1    4600 10450
@@
 F 0 "R9" H 5081 9896 50  0000 R CNN
 F 1 "10k" H 5081 9805 50  0000 R CNN
-F 2 "Resistor_SMD:R_0805_2012Metric" V 5080 9850 50  0001 C CNN
+F 2 "Resistor_SMD:R_0805_2012Metric_Pad1.15x1.40mm_HandSolder" V 5080 9850 50  0001 C CNN
 F 3 "~" H 5150 9850 50  0001 C CNN
 	1    5150 9850
@@
 F 0 "R10" H 5431 9896 50  0000 R CNN
 F 1 "10k" H 5431 9805 50  0000 R CNN
-F 2 "Resistor_SMD:R_0805_2012Metric" V 5430 9850 50  0001 C CNN
+F 2 "Resistor_SMD:R_0805_2012Metric_Pad1.15x1.40mm_HandSolder" V 5430 9850 50  0001 C CNN
 F 3 "~" H 5500 9850 50  0001 C CNN
 	1    5500 9850
@@
 F 0 "R12" H 6420 4746 50  0000 L CNN
 F 1 "47k" H 6420 4655 50  0000 L CNN
-F 2 "Resistor_SMD:R_0805_2012Metric" V 6280 4700 50  0001 C CNN
+F 2 "Resistor_SMD:R_0805_2012Metric_Pad1.15x1.40mm_HandSolder" V 6280 4700 50  0001 C CNN
 F 3 "~" H 6350 4700 50  0001 C CNN
 	1    6350 4700
@@
 F 0 "R11" H 6420 6496 50  0000 L CNN
 F 1 "47k" H 6420 6405 50  0000 L CNN
-F 2 "Resistor_SMD:R_0805_2012Metric" V 6280 6450 50  0001 C CNN
+F 2 "Resistor_SMD:R_0805_2012Metric_Pad1.15x1.40mm_HandSolder" V 6280 6450 50  0001 C CNN
 F 3 "~" H 6350 6450 50  0001 C CNN
 	1    6350 6450
@@
 F 0 "R13" H 8480 8596 50  0000 R CNN
 F 1 "10k" H 8480 8505 50  0000 R CNN
-F 2 "Resistor_SMD:R_0805_2012Metric" V 8480 8550 50  0001 C CNN
+F 2 "Resistor_SMD:R_0805_2012Metric_Pad1.15x1.40mm_HandSolder" V 8480 8550 50  0001 C CNN
 F 3 "~" H 8550 8550 50  0001 C CNN
 	1    8550 8550
@@
 F 0 "R14" H 8480 9296 50  0000 R CNN
 F 1 "10k" H 8480 9205 50  0000 R CNN
-F 2 "Resistor_SMD:R_0805_2012Metric" V 8480 9250 50  0001 C CNN
+F 2 "Resistor_SMD:R_0805_2012Metric_Pad1.15x1.40mm_HandSolder" V 8480 9250 50  0001 C CNN
 F 3 "~" H 8550 9250 50  0001 C CNN
 	1    8550 9250
@@
 F 0 "R15" H 8670 4746 50  0000 L CNN
 F 1 "47k" H 8670 4655 50  0000 L CNN
-F 2 "Resistor_SMD:R_0805_2012Metric" V 8530 4700 50  0001 C CNN
+F 2 "Resistor_SMD:R_0805_2012Metric_Pad1.15x1.40mm_HandSolder" V 8530 4700 50  0001 C CNN
 F 3 "~" H 8600 4700 50  0001 C CNN
 	1    8600 4700
@@
 F 0 "R16" H 8670 6496 50  0000 L CNN
 F 1 "47k" H 8670 6405 50  0000 L CNN
-F 2 "Resistor_SMD:R_0805_2012Metric" V 8530 6450 50  0001 C CNN
+F 2 "Resistor_SMD:R_0805_2012Metric_Pad1.15x1.40mm_HandSolder" V 8530 6450 50  0001 C CNN
 F 3 "~" H 8600 6450 50  0001 C CNN
 	1    8600 6450
@@
 F 0 "R18" V 11943 2850 50  0000 C CNN
 F 1 "1k" V 12034 2850 50  0000 C CNN
-F 2 "Resistor_SMD:R_0805_2012Metric" V 12080 2850 50  0001 C CNN
+F 2 "Resistor_SMD:R_0805_2012Metric_Pad1.15x1.40mm_HandSolder" V 12080 2850 50  0001 C CNN
 F 3 "~" H 12150 2850 50  0001 C CNN
 	1    12150 2850
@@
 F 0 "R19" V 11943 4900 50  0000 C CNN
 F 1 "1k" V 12034 4900 50  0000 C CNN
-F 2 "Resistor_SMD:R_0805_2012Metric" V 12080 4900 50  0001 C CNN
+F 2 "Resistor_SMD:R_0805_2012Metric_Pad1.15x1.40mm_HandSolder" V 12080 4900 50  0001 C CNN
 F 3 "~" H 12150 4900 50  0001 C CNN
 	1    12150 4900
@@
 F 0 "R20" H 12550 3200 50  0000 R CNN
 F 1 "4.7k" H 12600 3100 50  0000 R CNN
-F 2 "Resistor_SMD:R_0805_2012Metric" V 12330 3150 50  0001 C CNN
+F 2 "Resistor_SMD:R_0805_2012Metric_Pad1.15x1.40mm_HandSolder" V 12330 3150 50  0001 C CNN
 F 3 "~" H 12400 3150 50  0001 C CNN
 	1    12400 3150
@@
 F 0 "R21" H 12550 5250 50  0000 R CNN
 F 1 "4.7k" H 12600 5150 50  0000 R CNN
-F 2 "Resistor_SMD:R_0805_2012Metric" V 12330 5200 50  0001 C CNN
+F 2 "Resistor_SMD:R_0805_2012Metric_Pad1.15x1.40mm_HandSolder" V 12330 5200 50  0001 C CNN
 F 3 "~" H 12400 5200 50  0001 C CNN
 	1    12400 5200
@@
 F 0 "R22" H 12731 2446 50  0000 R CNN
 F 1 "1k" H 12731 2355 50  0000 R CNN
-F 2 "Resistor_SMD:R_0805_2012Metric" V 12730 2400 50  0001 C CNN
+F 2 "Resistor_SMD:R_0805_2012Metric_Pad1.15x1.40mm_HandSolder" V 12730 2400 50  0001 C CNN
 F 3 "~" H 12800 2400 50  0001 C CNN
 	1    12800 2400
@@
 F 0 "R23" H 12731 4496 50  0000 R CNN
 F 1 "1k" H 12731 4405 50  0000 R CNN
-F 2 "Resistor_SMD:R_0805_2012Metric" V 12730 4450 50  0001 C CNN
+F 2 "Resistor_SMD:R_0805_2012Metric_Pad1.15x1.40mm_HandSolder" V 12730 4450 50  0001 C CNN
 F 3 "~" H 12800 4450 50  0001 C CNN
 	1    12800 4450
@@
 F 0 "R28" H 15700 5400 50  0000 R CNN
 F 1 "4.7k" H 15750 5300 50  0000 R CNN
-F 2 "Resistor_SMD:R_0805_2012Metric" V 15480 5350 50  0001 C CNN
+F 2 "Resistor_SMD:R_0805_2012Metric_Pad1.15x1.40mm_HandSolder" V 15480 5350 50  0001 C CNN
 F 3 "~" H 15550 5350 50  0001 C CNN
 	1    15550 5350
@@
 F 0 "C1" H 1665 5046 50  0000 L CNN
 F 1 "100n" H 1665 4955 50  0000 L CNN
-F 2 "Capacitor_SMD:C_0805_2012Metric" H 1588 4850 50  0001 C CNN
+F 2 "Capacitor_SMD:C_0805_2012Metric_Pad1.15x1.40mm_HandSolder" H 1588 4850 50  0001 C CNN
 F 3 "~" H 1550 5000 50  0001 C CNN
 	1    1550 5000
@@
 F 0 "C9" H 1665 5996 50  0000 L CNN
 F 1 "100n" H 1665 5905 50  0000 L CNN
-F 2 "Capacitor_SMD:C_0805_2012Metric" H 1588 5800 50  0001 C CNN
+F 2 "Capacitor_SMD:C_0805_2012Metric_Pad1.15x1.40mm_HandSolder" H 1588 5800 50  0001 C CNN
 F 3 "~" H 1550 5950 50  0001 C CNN
 	1    1550 5950
@@
 F 0 "C2" H 2065 10196 50  0000 L CNN
 F 1 "100n" H 2065 10105 50  0000 L CNN
-F 2 "Capacitor_SMD:C_0805_2012Metric" H 1988 10000 50  0001 C CNN
+F 2 "Capacitor_SMD:C_0805_2012Metric_Pad1.15x1.40mm_HandSolder" H 1988 10000 50  0001 C CNN
 F 3 "~" H 1950 10150 50  0001 C CNN
 	1    1950 10150
@@
 F 0 "C10" H 2815 9696 50  0000 L CNN
 F 1 "10p" H 2815 9605 50  0000 L CNN
-F 2 "Capacitor_SMD:C_0805_2012Metric" H 2738 9500 50  0001 C CNN
+F 2 "Capacitor_SMD:C_0805_2012Metric_Pad1.15x1.40mm_HandSolder" H 2738 9500 50  0001 C CNN
 F 3 "~" H 2700 9650 50  0001 C CNN
 	1    2700 9650
@@
 F 0 "C5" H 7715 8646 50  0000 L CNN
 F 1 "100n" H 7715 8555 50  0000 L CNN
-F 2 "Capacitor_SMD:C_0805_2012Metric" H 7638 8450 50  0001 C CNN
+F 2 "Capacitor_SMD:C_0805_2012Metric_Pad1.15x1.40mm_HandSolder" H 7638 8450 50  0001 C CNN
 F 3 "~" H 7600 8600 50  0001 C CNN
 	1    7600 8600
@@
 F 0 "C4" H 7765 10346 50  0000 L CNN
 F 1 "20pF" H 7765 10255 50  0000 L CNN
-F 2 "Capacitor_SMD:C_0805_2012Metric" H 7688 10150 50  0001 C CNN
+F 2 "Capacitor_SMD:C_0805_2012Metric_Pad1.15x1.40mm_HandSolder" H 7688 10150 50  0001 C CNN
 F 3 "~" H 7650 10300 50  0001 C CNN
 	1    7650 10300
@@
 F 0 "C6" H 8265 10346 50  0000 L CNN
 F 1 "20pF" H 8265 10255 50  0000 L CNN
-F 2 "Capacitor_SMD:C_0805_2012Metric" H 8188 10150 50  0001 C CNN
+F 2 "Capacitor_SMD:C_0805_2012Metric_Pad1.15x1.40mm_HandSolder" H 8188 10150 50  0001 C CNN
 F 3 "~" H 8150 10300 50  0001 C CNN
 	1    8150 10300
@@
 F 0 "C13" H 10865 9496 50  0000 L CNN
 F 1 "100n" H 10865 9405 50  0000 L CNN
-F 2 "Capacitor_SMD:C_0805_2012Metric" H 10788 9300 50  0001 C CNN
+F 2 "Capacitor_SMD:C_0805_2012Metric_Pad1.15x1.40mm_HandSolder" H 10788 9300 50  0001 C CNN
 F 3 "~" H 10750 9450 50  0001 C CNN
 	1    10750 9450
@@
 F 0 "C14" H 10865 10446 50  0000 L CNN
 F 1 "100n" H 10865 10355 50  0000 L CNN
-F 2 "Capacitor_SMD:C_0805_2012Metric" H 10788 10250 50  0001 C CNN
+F 2 "Capacitor_SMD:C_0805_2012Metric_Pad1.15x1.40mm_HandSolder" H 10788 10250 50  0001 C CNN
 F 3 "~" H 10750 10400 50  0001 C CNN
 	1    10750 10400
@@
 F 0 "C15" H 11315 9496 50  0000 L CNN
 F 1 "100n" H 11315 9405 50  0000 L CNN
-F 2 "Capacitor_SMD:C_0805_2012Metric" H 11238 9300 50  0001 C CNN
+F 2 "Capacitor_SMD:C_0805_2012Metric_Pad1.15x1.40mm_HandSolder" H 11238 9300 50  0001 C CNN
 F 3 "~" H 11200 9450 50  0001 C CNN
 	1    11200 9450
@@
 F 0 "C7" H 11315 10446 50  0000 L CNN
 F 1 "100n" H 11315 10355 50  0000 L CNN
-F 2 "Capacitor_SMD:C_0805_2012Metric" H 11238 10250 50  0001 C CNN
+F 2 "Capacitor_SMD:C_0805_2012Metric_Pad1.15x1.40mm_HandSolder" H 11238 10250 50  0001 C CNN
 F 3 "~" H 11200 10400 50  0001 C CNN
 	1    11200 10400
@@
 F 0 "C11" H 12915 9496 50  0000 L CNN
 F 1 "100n" H 12915 9405 50  0000 L CNN
-F 2 "Capacitor_SMD:C_0805_2012Metric" H 12838 9300 50  0001 C CNN
+F 2 "Capacitor_SMD:C_0805_2012Metric_Pad1.15x1.40mm_HandSolder" H 12838 9300 50  0001 C CNN
 F 3 "~" H 12800 9450 50  0001 C CNN
 	1    12800 9450
