File: stepper/stepper.kicad_pcb (KiCad board)
At the start: 2 copper layers, 50 x 25 mm, 19 parts, among them J1 VDD_IN, J2 In, J3 Jumpers, J4 Stepper

Commit message: cosmetic changes
Other:
- board text added: "protopit.eu"
