File: led_board/led_board.kicad_pcb (KiCad board)
At the start: 2 copper layers, 180 x 25 mm, 138 parts, among them J1 Power

Commit message: properly space leds on pcb
Parts:
- moved R3 24.6 mm to (197.0, 36.0)
- moved R1 15.7 mm to (129.0, 46.0)
- moved D49 1.00 mm to (119.0, 63.0)
- moved D50 1.00 mm to (111.0, 63.0)
- moved D51 1.00 mm to (103.0, 63.0)
- moved D52 1.00 mm to (95.0, 63.0)
- moved D53 1.00 mm to (87.0, 63.0)
- moved D54 1.00 mm to (79.0, 63.0)
- moved D55 1.00 mm to (71.0, 63.0)
- moved D56 1.00 mm to (63.0, 63.0)
- moved D57 1.00 mm to (119.0, 58.0)
- moved D58 1.00 mm to (111.0, 58.0)
- moved D59 1.00 mm to (103.0, 58.0)
- moved D60 1.00 mm to (95.0, 58.0)
- moved D61 1.00 mm to (87.0, 58.0)
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Routing:
- net Net-(D40-Pad1): track 0.00 -> 18.1 mm
- net Net-(D48-Pad1): track 0.00 -> 17.3 mm
- net /VPOS: track 96.7 -> 83.8 mm
- net /VNEG_A: track 170.8 -> 174.5 mm
- net Net-(D9-Pad2): track 3.02 -> 0.00 mm
- net Net-(D17-Pad2): track 3.12 -> 0.11 mm
- added copper zone on F.Cu, net /VPOS

Commit message: rearrange led board pcb
Parts:
- moved H2 248.0 mm to (354.0, 66.5)
- moved H4 174.5 mm to (279.0, 66.5)
- moved D113 76.0 mm to (269.1, 75.0)
- moved D114 76.0 mm to (261.1, 75.0)
- moved D115 76.0 mm to (253.1, 75.0)
- moved D116 76.0 mm to (245.1, 75.0)
- moved D117 76.0 mm to (237.1, 75.0)
- moved D118 76.0 mm to (229.1, 75.0)
- moved D119 76.0 mm to (221.1, 75.0)
- moved D120 76.0 mm to (213.1, 75.0)
- moved D121 76.0 mm to (269.1, 70.0)
- moved D122 76.0 mm to (261.1, 70.0)
- moved D123 76.0 mm to (253.1, 70.0)
- moved D124 76.0 mm to (245.1, 70.0)
- moved D125 76.0 mm to (237.1, 70.0)
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Connections:
- D1 pad 2: /VPOS -> Net-(D1-Pad2)
- D9 pad 2: Net-(D9-Pad2) -> /VPOS
- R1 pad 1: /VPOS -> Net-(D1-Pad2)
- R1 pad 2: Net-(D9-Pad2) -> /VPOS
Routing:
- net /VNEG_B: track 220.6 -> 658.3 mm
- net /VNEG_A: track 174.5 -> 606.0 mm
- net /VPOS: track 83.8 -> 288.1 mm
- net Net-(D16-Pad1): track 0.00 -> 17.0 mm
- net Net-(D17-Pad2): track 0.11 -> 16.9 mm
- net Net-(D1-Pad2): track 0.00 -> 4.11 mm
- net Net-(D41-Pad2): track 0.00 -> 3.97 mm
