File: boards/standalone/dimmable_psu/dimmable_psu.kicad_sch (KiCad schematic)
At the start: 0 parts

Commit message: add buck converter ic
Parts:
- added U1: TPS92640, Package_SO:HTSSOP-14-1EP_4.4x5mm_P0.65mm_EP3.4x5mm_Mask3x3.1mm, symbol ti_reg:TPS92640
Changed lines of the file:
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@@
-(kicad_sch (version 20200310) (host eeschema "unknown")
-(  page "A4")
-  (symbol_instances)
+(kicad_sch (version 20210126) (generator eeschema)
+  (paper "A4")
+  (symbol (lib_id "ti_reg:TPS92640") (at 134.62 81.28 0) (unit 1)
+    (in_bom yes) (on_board yes)
+    (property "Reference" "U1" (id 0) (at 135.89 67.31 0))
+    (property "Value" "TPS92640" (id 1) (at 135.89 69.85 0))
+    (property "Footprint" "Package_SO:HTSSOP-14-1EP_4.4x5mm_P0.65mm_EP3.4x5mm_Mask3x3.1mm" (id 2) (at 107.95 92.71 0)
+      (effects (font (size 1.27 1.27)) (justify left) hide)
+    )
+    (property "Datasheet" "https://www.ti.com/lit/ds/symlink/tps92640.pdf" (id 3) (at 134.62 67.31 0)
+      (effects (font (size 1.27 1.27)) hide)
+    )
+    (property "shop" "https://bg.farnell.com/texas-instruments/tps92640pwp-nopb/driver-led-1mhz-1a-2ohm-14tssop/dp/3119220?st=tps92640" (id 4) (at 142.24 63.5 0)
+      (effects (font (size 1.27 1.27)) hide)
+    )
+    (pin "1")
+    (pin "2")
+    (pin "3")
+    (pin "4")
+    (pin "5")
+    (pin "6")
+    (pin "7")
+    (pin "8")
+    (pin "9")
+    (pin "10")
+    (pin "11")
+    (pin "12")
+    (pin "13")
+    (pin "14")
+  )
+  (sheet_instances
+    (path "/" (page "1"))
+  )
+  (symbol_instances
+    (path "/1e85445e-8800-4362-acdc-87d9808fb140"
+      (reference "U1") (unit 1) (value "TPS92640") (footprint "Package_SO:HTSSOP-14-1EP_4.4x5mm_P0.65mm_EP3.4x5mm_Mask3x3.1mm")
+    )
+  )
 )
