File: boards/standalone/dimmable_psu/dimmable_psu.kicad_sch (KiCad schematic)
At the start: 82 parts, among them J1 DIM_IN, J2 PWM_IN, J3 POWER, J4 POWER_OUT, Q1 2N7002, Q2 IRF540N, Q3 IRF540N, U1 LM324, U2 LMC7660, U3 TPS92640

Commit message: arrange power-side stuff
Parts:
- gave numbers to parts that had none: 4
Connections:
- net GND: now also J3.2 (Pin_2); no longer J3.1 (Pin_1)
- net VPP: now also J3.1 (Pin_1); no longer J3.2 (Pin_2)
- net POWER_JUN: now reaches C16.1, L1.1, Q2.3 (S), Q3.2 (D), TP8.1, U3.13 (SW)
- net OUT+: now reaches C18.1, L1.2, R19.1, R24.1
- net OUT+: now also J4.2 (Pin_2); no longer J4.1 (Pin_1)
- net CSENSE: now reaches R24.2, U3.9 (CSENSE)
- net CSENSE: now also R25.2; no longer R25.1
- net at D5.1 (K), R9.1: now also JP2.1 (A); no longer JP2.2 (B)
- net OUT-: now reaches C18.2, R26.1, R27.1, R28.1
- net OUT-: now also J4.1 (Pin_1), R25.1; no longer J4.2 (Pin_2), R25.2
- net at D5.2 (A), JP1.2 (B), U1.1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: now also JP2.2 (B); no longer JP2.1 (A)
Other:
- moved on the sheet: J3, R25
Changed lines of the file:
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@@
+    (effects (font (size 1.27 1.27)) (justify right bottom))
+  )
+  (label "POWER_JUN" (at 318.135 77.47 180)
+    (effects (font (size 1.27 1.27)) (justify right bottom))
+  )
+  (label "CSENSE" (at 336.55 135.89 180)
+    (effects (font (size 1.27 1.27)) (justify right bottom))
+  )
+  (label "OUT+" (at 367.665 77.47 180)
+    (effects (font (size 1.27 1.27)) (justify right bottom))
+  )
+  (label "OUT-" (at 367.665 92.71 180)
     (effects (font (size 1.27 1.27)) (justify right bottom))
   )
@@
     (pin "2")
   )
-  (symbol (lib_id "Device:R") (at 353.06 135.89 90) (unit 1)
-    (in_bom yes) (on_board yes)
-    (property "Reference" "R25" (id 0) (at 354.203 136.017 90)
-      (effects (font (size 1.27 1.27)) (justify left))
-    )
-    (property "Value" "10" (id 1) (at 354.965 138.43 90)
-      (effects (font (size 1.27 1.27)) (justify left))
-    )
-    (property "Footprint" "Resistor_THT:R_Axial_DIN0309_L9.0mm_D3.2mm_P12.70mm_Horizontal" (id 2) (at 353.06 137.668 90)
+  (symbol (lib_id "Device:R") (at 353.06 135.89 270) (unit 1)
+    (in_bom yes) (on_board yes)
+    (property "Reference" "R25" (id 0) (at 351.917 135.763 90)
+      (effects (font (size 1.27 1.27)) (justify left))
+    )
+    (property "Value" "10" (id 1) (at 351.155 133.35 90)
+      (effects (font (size 1.27 1.27)) (justify left))
+    )
+    (property "Footprint" "Resistor_THT:R_Axial_DIN0309_L9.0mm_D3.2mm_P12.70mm_Horizontal" (id 2) (at 353.06 134.112 90)
       (effects (font (size 1.27 1.27)) hide)
     )
@@
   (symbol (lib_id "Mechanical:MountingHole_Pad") (at 372.745 255.905 0) (unit 1)
     (in_bom yes) (on_board yes)
-    (property "Reference" "H?" (id 0) (at 371.475 251.46 0)
+    (property "Reference" "H1" (id 0) (at 371.475 251.46 0)
       (effects (font (size 1.27 1.27)) (justify left))
     )
@@
   (symbol (lib_id "Mechanical:MountingHole_Pad") (at 377.19 255.905 0) (unit 1)
     (in_bom yes) (on_board yes)
-    (property "Reference" "H?" (id 0) (at 375.92 251.46 0)
+    (property "Reference" "H2" (id 0) (at 375.92 251.46 0)
       (effects (font (size 1.27 1.27)) (justify left))
     )
@@
   (symbol (lib_id "Mechanical:MountingHole_Pad") (at 381.635 255.905 0) (unit 1)
     (in_bom yes) (on_board yes)
-    (property "Reference" "H?" (id 0) (at 380.365 251.46 0)
+    (property "Reference" "H3" (id 0) (at 380.365 251.46 0)
       (effects (font (size 1.27 1.27)) (justify left))
     )
@@
   (symbol (lib_id "Mechanical:MountingHole_Pad") (at 386.08 255.905 0) (unit 1)
     (in_bom yes) (on_board yes)
-    (property "Reference" "H?" (id 0) (at 384.81 251.46 0)
+    (property "Reference" "H4" (id 0) (at 384.81 251.46 0)
       (effects (font (size 1.27 1.27)) (justify left))
     )
@@
     (pin "2")
   )
-  (symbol (lib_id "Jumper:Jumper_2_Bridged") (at 111.76 43.18 0) (unit 1)
+  (symbol (lib_id "Jumper:Jumper_2_Bridged") (at 111.76 43.18 0) (mirror y) (unit 1)
     (in_bom yes) (on_board yes)
     (property "Reference" "JP2" (id 0) (at 111.76 38.1 0))
@@
     (pin "2")
   )
-  (symbol (lib_id "Connector_Generic:Conn_01x02") (at 43.18 229.87 180) (unit 1)
-    (in_bom yes) (on_board yes)
-    (property "Reference" "J3" (id 0) (at 40.64 229.87 0)
-      (effects (font (size 1.27 1.27)) (justify left))
-    )
-    (property "Value" "POWER" (id 1) (at 40.64 227.33 0)
-      (effects (font (size 1.27 1.27)) (justify left))
-    )
-    (property "Footprint" "wago:2061-602" (id 2) (at 43.18 229.87 0)
-      (effects (font (size 1.27 1.27)) hide)
-    )
-    (property "Datasheet" "~" (id 3) (at 43.18 229.87 0)
-      (effects (font (size 1.27 1.27)) hide)
-    )
-    (pin "1")
-    (pin "2")
-  )
-  (symbol (lib_id "Connector_Generic:Conn_01x02") (at 379.73 77.47 0) (unit 1)
-    (in_bom yes) (on_board yes)
-    (property "Reference" "J4" (id 0) (at 382.27 77.47 0)
-      (effects (font (size 1.27 1.27)) (justify left))
-    )
-    (property "Value" "POWER_OUT" (id 1) (at 382.27 80.01 0)
-      (effects (font (size 1.27 1.27)) (justify left))
-    )
-    (property "Footprint" "wago:2061-602" (id 2) (at 379.73 77.47 0)
-      (effects (font (size 1.27 1.27)) hide)
-    )
-    (property "Datasheet" "~" (id 3) (at 379.73 77.47 0)
+  (symbol (lib_id "Connector_Generic:Conn_01x02") (at 43.18 227.33 0) (mirror y) (unit 1)
+    (in_bom yes) (on_board yes)
+    (property "Reference" "J3" (id 0) (at 40.64 227.33 0)
+      (effects (font (size 1.27 1.27)) (justify left))
+    )
+    (property "Value" "POWER" (id 1) (at 40.64 229.87 0)
+      (effects (font (size 1.27 1.27)) (justify left))
+    )
+    (property "Footprint" "wago:2061-602" (id 2) (at 43.18 227.33 0)
+      (effects (font (size 1.27 1.27)) hide)
+    )
+    (property "Datasheet" "~" (id 3) (at 43.18 227.33 0)
+      (effects (font (size 1.27 1.27)) hide)
+    )
+    (pin "1")
+    (pin "2")
+  )
+  (symbol (lib_id "Connector_Generic:Conn_01x02") (at 379.73 80.01 0) (mirror x) (unit 1)
+    (in_bom yes) (on_board yes)
+    (property "Reference" "J4" (id 0) (at 382.27 80.01 0)
+      (effects (font (size 1.27 1.27)) (justify left))
+    )
+    (property "Value" "POWER_OUT" (id 1) (at 382.27 77.47 0)
+      (effects (font (size 1.27 1.27)) (justify left))
+    )
+    (property "Footprint" "wago:2061-602" (id 2) (at 379.73 80.01 0)
+      (effects (font (size 1.27 1.27)) hide)
+    )
+    (property "Datasheet" "~" (id 3) (at 379.73 80.01 0)
       (effects (font (size 1.27 1.27)) hide)
     )
@@
     )
     (path "/023ebd38-5f1e-458e-be61-bb156e5173ae"
-      (reference "H?") (unit 1) (value "MountingHole_Pad") (footprint "MountingHole:MountingHole_3.2mm_M3_Pad")
+      (reference "H1") (unit 1) (value "MountingHole_Pad") (footprint "MountingHole:MountingHole_3.2mm_M3_Pad")
+    )
+    (path "/edab61e6-910c-4e8e-95df-adcb0437978a"
+      (reference "H2") (unit 1) (value "MountingHole_Pad") (footprint "MountingHole:MountingHole_3.2mm_M3_Pad")
     )
     (path "/18a07627-8ae3-4b6b-89bb-064a36bbb40d"
-      (reference "H?") (unit 1) (value "MountingHole_Pad") (footprint "MountingHole:MountingHole_3.2mm_M3_Pad")
+      (reference "H3") (unit 1) (value "MountingHole_Pad") (footprint "MountingHole:MountingHole_3.2mm_M3_Pad")
     )
     (path "/dc36ab86-8ce5-42ab-87c0-719642f09dff"
-      (reference "H?") (unit 1) (value "MountingHole_Pad") (footprint "MountingHole:MountingHole_3.2mm_M3_Pad")
-    )
-    (path "/edab61e6-910c-4e8e-95df-adcb0437978a"
-      (reference "H?") (unit 1) (value "MountingHole_Pad") (footprint "MountingHole:MountingHole_3.2mm_M3_Pad")
+      (reference "H4") (unit 1) (value "MountingHole_Pad") (footprint "MountingHole:MountingHole_3.2mm_M3_Pad")
     )
     (path "/d48847fd-ac00-4036-90e4-501d8884232c"
