File: boards/standalone/dimmable_psu/dimmable_psu.kicad_pcb (KiCad board)
At the start: 0 parts

Commit message: final touches to dimmable psu schematic
Parts:
- added C1: 470n, Capacitor_SMD:C_0805_2012Metric_Pad1.18x1.45mm_HandSolder, F.Cu at (177.8, 71.2)
- added C10: 10µ, Capacitor_SMD:CP_Elec_5x5.4, F.Cu at (112.5, 108.8)
- added C11: 1n, Capacitor_SMD:C_0805_2012Metric_Pad1.18x1.45mm_HandSolder, F.Cu at (172.9, 71.2)
- added C12: 1µ, Capacitor_SMD:C_0805_2012Metric_Pad1.18x1.45mm_HandSolder, F.Cu at (133.0, 110.4)
- added C13: 100n, Capacitor_SMD:C_0805_2012Metric_Pad1.18x1.45mm_HandSolder, F.Cu at (155.6, 89.5)
- added C14: 470n, Capacitor_SMD:C_0805_2012Metric_Pad1.18x1.45mm_HandSolder, F.Cu at (163.5, 85.0)
- added C15: 100n, Capacitor_SMD:C_0805_2012Metric_Pad1.18x1.45mm_HandSolder, F.Cu at (143.0, 102.1)
- added C16: 100n, Capacitor_SMD:C_0805_2012Metric_Pad1.18x1.45mm_HandSolder, F.Cu at (150.6, 98.7)
- added C17: 2.2µ, Capacitor_SMD:C_0805_2012Metric_Pad1.18x1.45mm_HandSolder, F.Cu at (143.0, 105.1)
- added C18: 100uF, Capacitor_THT:CP_Radial_D12.5mm_P5.00mm, F.Cu at (152.1, 70.1)
- added C2: 470µ, Capacitor_THT:CP_Radial_D16.0mm_P7.50mm, F.Cu at (119.5, 152.0)
- added C3: 100n, Capacitor_SMD:C_0805_2012Metric_Pad1.18x1.45mm_HandSolder, F.Cu at (172.9, 74.3)
- added C4: 10µ, Capacitor_SMD:CP_Elec_5x5.4, F.Cu at (121.4, 108.8)
- added C5: 100n, Capacitor_SMD:C_0805_2012Metric_Pad1.18x1.45mm_HandSolder, F.Cu at (137.8, 107.4)
- added C6: 10µ, Capacitor_SMD:CP_Elec_5x5.4, F.Cu at (136.1, 102.4)
- added C7: 100n, Capacitor_SMD:C_0805_2012Metric_Pad1.18x1.45mm_HandSolder, F.Cu at (133.0, 107.4)
- added C8: 10p, Capacitor_SMD:C_0805_2012Metric_Pad1.18x1.45mm_HandSolder, F.Cu at (137.8, 110.4)
- added C9: 10µ, Capacitor_SMD:CP_Elec_5x5.4, F.Cu at (166.1, 72.9)
- added D1: D_Schottky_Trans, Diode_SMD:D_SOD-123, B.Cu at (98.5, 139.0)
- added D10: D_Schottky, Diode_SMD:D_SOD-123, F.Cu at (175.6, 68.1)
- added D2: D_Schottky_Trans, Diode_SMD:D_SOD-123, B.Cu at (96.5, 141.5)
- added D3: D_Schottky_Trans, Diode_SMD:D_SOD-123, B.Cu at (98.5, 131.0)
- added D4: D_Schottky_Trans, Diode_SMD:D_SOD-123, B.Cu at (96.5, 133.5)
- added D5: D, Diode_SMD:D_SOD-123, F.Cu at (150.1, 78.8)
- added D6: 15v, Diode_THT:D_DO-15_P12.70mm_Horizontal, F.Cu at (144.5, 136.0)
- added D7: D, Diode_SMD:D_SOD-123, F.Cu at (110.9, 113.9)
- added D8: D, Diode_SMD:D_SOD-123, F.Cu at (128.1, 114.3)
- added D9: 2.7v, Diode_THT:D_DO-15_P12.70mm_Horizontal, F.Cu at (135.5, 136.0)
- added J1: DIM_IN, wago:250-402, F.Cu at (102.5, 138.0)
- added J2: PWM_IN, wago:250-402, F.Cu at (102.5, 130.5)
- added J3: POWER, wago:2061-602, F.Cu at (100.0, 149.0)
- added J4: POWER_OUT, wago:2061-602, F.Cu at (204.0, 116.0)
- added JP1: AUTO_OFF, Connector_PinHeader_2.54mm:PinHeader_1x02_P2.54mm_Vertical, F.Cu at (133.0, 122.0)
- added JP2: ~ZERO_OFFSET, Connector_PinHeader_2.54mm:PinHeader_1x02_P2.54mm_Vertical, F.Cu at (122.8, 93.5)
- added L1: 100µH, inductors:L_Bourns_SRR1770, F.Cu at (105.5, 71.2)
- added Q1: 2N7002, Package_TO_SOT_SMD:SOT-23, F.Cu at (158.6, 85.8)
- added Q2: IRF540N, Package_TO_SOT_THT:TO-220-3_Vertical, F.Cu at (99.7, 108.0)
- added Q3: IRF540N, Package_TO_SOT_THT:TO-220-3_Vertical, F.Cu at (99.7, 114.0)
- added R1: 47k, Resistor_SMD:R_0805_2012Metric_Pad1.20x1.40mm_HandSolder, B.Cu at (103.5, 136.5)
- added R10: 22k, Potentiometer_THT:Potentiometer_Bourns_3296Y_Vertical, F.Cu at (169.7, 65.0)
- added R11: 10k, Resistor_SMD:R_0805_2012Metric_Pad1.20x1.40mm_HandSolder, F.Cu at (155.6, 92.5)
- added R12: 22k, Potentiometer_THT:Potentiometer_Bourns_3296Y_Vertical, F.Cu at (141.8, 87.3)
- added R13: 100, Resistor_SMD:R_0805_2012Metric_Pad1.20x1.40mm_HandSolder, F.Cu at (182.5, 70.8)
- added R14: rudim1, Resistor_SMD:R_0805_2012Metric_Pad1.20x1.40mm_HandSolder, F.Cu at (186.6, 64.5)
- added R15: rudim2, Resistor_SMD:R_0805_2012Metric_Pad1.20x1.40mm_HandSolder, F.Cu at (168.2, 87.0)
- added R16: 1.2k, Resistor_THT:R_Axial_DIN0309_L9.0mm_D3.2mm_P12.70mm_Horizontal, F.Cu at (131.0, 152.0)
- added R17: rudim3, Resistor_SMD:R_0805_2012Metric_Pad1.20x1.40mm_HandSolder, F.Cu at (172.9, 77.2)
- added R18: 10k, Resistor_SMD:R_0805_2012Metric_Pad1.20x1.40mm_HandSolder, F.Cu at (172.7, 80.2)
- added R19: 150k, Resistor_SMD:R_0805_2012Metric_Pad1.20x1.40mm_HandSolder, F.Cu at (180.9, 67.9)
- added R2: 100k, Resistor_SMD:R_0805_2012Metric_Pad1.20x1.40mm_HandSolder, B.Cu at (97.0, 128.5)
- added R20: 22k, Potentiometer_THT:Potentiometer_Bourns_3296Y_Vertical, F.Cu at (153.1, 82.5)
- added R21: ron, Resistor_SMD:R_0805_2012Metric_Pad1.20x1.40mm_HandSolder, F.Cu at (160.4, 92.4)
- added R22: rhg, Resistor_SMD:R_0805_2012Metric_Pad1.20x1.40mm_HandSolder, F.Cu at (155.4, 98.7)
- added R23: rlg, Resistor_SMD:R_0805_2012Metric_Pad1.20x1.40mm_HandSolder, F.Cu at (160.4, 89.5)
- added R24: 150, Resistor_THT:R_Axial_DIN0309_L9.0mm_D3.2mm_P12.70mm_Horizontal, F.Cu at (130.7, 83.0)
- added R25: 10, Resistor_THT:R_Axial_DIN0309_L9.0mm_D3.2mm_P12.70mm_Horizontal, F.Cu at (147.8, 102.0)
- added R26: 0.2, Resistor_THT:R_Axial_DIN0309_L9.0mm_D3.2mm_P12.70mm_Horizontal, F.Cu at (111.2, 88.8)
- added R27: 0.2, Resistor_THT:R_Axial_DIN0309_L9.0mm_D3.2mm_P12.70mm_Horizontal, F.Cu at (111.2, 84.0)
- added R28: 0.2, Resistor_THT:R_Axial_DIN0309_L9.0mm_D3.2mm_P12.70mm_Horizontal, F.Cu at (98.0, 101.7)
- added R29: 10M, Resistor_SMD:R_0805_2012Metric_Pad1.20x1.40mm_HandSolder, B.Cu at (97.0, 136.5)
- added R3: 10k, Resistor_SMD:R_0805_2012Metric_Pad1.20x1.40mm_HandSolder, F.Cu at (133.4, 113.3)
- added R4: 22k, Potentiometer_THT:Potentiometer_Bourns_3296Y_Vertical, F.Cu at (128.6, 100.9)
- added R5: 1k, Resistor_SMD:R_0805_2012Metric_Pad1.20x1.40mm_HandSolder, F.Cu at (138.1, 113.3)
- added R6: 1k, Resistor_SMD:R_0805_2012Metric_Pad1.20x1.40mm_HandSolder, B.Cu at (103.5, 128.5)
- added R7: 100k, Resistor_SMD:R_0805_2012Metric_Pad1.20x1.40mm_HandSolder, F.Cu at (177.7, 74.2)
- added R8: 750, Resistor_THT:R_Axial_DIN0309_L9.0mm_D3.2mm_P12.70mm_Horizontal, F.Cu at (140.0, 152.0)
- added R9: 10k, Resistor_SMD:R_0805_2012Metric_Pad1.20x1.40mm_HandSolder, F.Cu at (147.8, 105.0)
- added TP1: TestPoint, TestPoint:TestPoint_THTPad_D2.0mm_Drill1.0mm, F.Cu at (151.8, 116.6)
- added TP2: TestPoint, TestPoint:TestPoint_THTPad_D2.0mm_Drill1.0mm, F.Cu at (147.7, 116.6)
- added TP3: TestPoint, TestPoint:TestPoint_THTPad_D2.0mm_Drill1.0mm, F.Cu at (147.7, 120.7)
- added TP4: TestPoint, TestPoint:TestPoint_THTPad_D2.0mm_Drill1.0mm, F.Cu at (143.7, 119.5)
- added TP5: TestPoint, TestPoint:TestPoint_THTPad_D2.0mm_Drill1.0mm, F.Cu at (152.4, 112.5)
- added TP6: TestPoint, TestPoint:TestPoint_THTPad_D2.0mm_Drill1.0mm, F.Cu at (156.5, 112.5)
- added TP7: TestPoint, TestPoint:TestPoint_THTPad_D2.0mm_Drill1.0mm, F.Cu at (148.4, 112.5)
- added TP8: TestPoint, TestPoint:TestPoint_THTPad_D2.0mm_Drill1.0mm, F.Cu at (143.7, 115.5)
- added U1: LM324, Package_SO:SO-14_3.9x8.65mm_P1.27mm, F.Cu at (120.0, 128.0)
- added U2: LMC7660, Package_SO:SOIC-8_3.9x4.9mm_P1.27mm, B.Cu at (133.0, 144.0)
- added U3: TPS92640, Package_SO:HTSSOP-14-1EP_4.4x5mm_P0.65mm_EP3.4x5mm_Mask3x3.1mm, F.Cu at (138.1, 95.0)
Routing:
- net GND: track 0.00 -> 42.5 mm
- net VPP: track 0.00 -> 24.2 mm
- net /PWM_IN: track 0.00 -> 10.8 mm
- net /DIM_IN: track 0.00 -> 10.8 mm
Other:
- copper layers 0 -> 2
