File: boards/standalone/dimmable_psu/dimmable_psu.kicad_pcb (KiCad board)
At the start: 2 copper layers, 85 x 50 mm, 87 parts, among them J1 DIM_IN, J2 PWM_IN, J3 POWER, J4 POWER_OUT, Q1 2N7002, Q2 BST52, Q3 BST52, Q4 IRF540N, Q5 IRF540N, SW1 SW_DIP_SPLIT_x02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

Commit message: rearrange
Parts:
- moved R27 21.8 mm to (61.1, 38.5), turned to 0 degrees
- moved C24 16.6 mm to (49.8, 22.6), turned to 90 degrees
- moved R28 14.0 mm to (61.1, 34.5), turned to 0 degrees
- moved R26 13.4 mm to (61.1, 22.5), turned to 0 degrees
- moved R25 9.31 mm to (61.1, 26.5), turned to 0 degrees
- moved J4 8.01 mm to (68.5, 14.0)
- moved H2 8.00 mm to (73.0, 4.00)
- moved H3 8.00 mm to (73.0, 46.0)
- moved R22 8.00 mm to (36.2, 19.0), turned to -90 degrees
- moved R29 6.63 mm to (61.1, 30.5), turned to 0 degrees
- moved C17 4.07 mm to (35.5, 15.0)
- turned Q3 to 90 degrees
Connections:
- J4 pad 1: /OUT- -> /OUT+
- J4 pad 2: /OUT+ -> /OUT-
Routing:
- net /CSENSE: track 28.0 -> 53.3 mm
- net VDD: track 71.1 -> 79.4 mm, vias 2 -> 3
- net /VOUT_SENSE: track 65.2 -> 58.6 mm
- net Net-(C19-Pad1): track 9.09 -> 11.8 mm
- net /VNEGREF: track 15.1 -> 15.0 mm, vias 2 -> 1
- net GND: vias 235 -> 119
- added copper zone on B.Cu, net /OUT-
Other:
- board size 85 x 50 mm -> 77 x 50 mm
