File: boards/bus_modules/pwm/pwm.kicad_sch (KiCad schematic)
At the start: 60 parts, among them J10 PASSIVE_OUT, J11 VPP, J12 OUT, J13 VPP, J14 OUT, J15 VPP, J16 PASSIVE_OUT, J17 VPP, J18 OUT, J19 VPP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

Commit message: random cosmetic stuff
Other:
- note added: "FIXME: this buck converter has VDD <= 5.5v?!"
