File: boards/bundled_esp/pwm_controller/pwm_controller.kicad_sch (KiCad schematic)
At the start: 64 parts

Commit message: this commit is vomit
Parts:
- removed C? (x2): 100n, Capacitor_SMD:C_0805_2012Metric_Pad1.18x1.45mm_HandSolder, symbol Device:C
- removed C? (x3): 10µ, Capacitor_SMD:CP_Elec_5x5.4, symbol Device:C_Polarized
- removed C? (x2): x, symbol Device:C
- removed C?: 100n, Capacitor_SMD:C_0805_2012Metric_Pad1.15x1.40mm_HandSolder, symbol Device:C
- removed C?: 10p, Capacitor_SMD:C_0805_2012Metric_Pad1.18x1.45mm_HandSolder, symbol Device:C
- removed C?: 10p, Capacitor_SMD:C_0805_2012Metric_Pad1.15x1.40mm_HandSolder, symbol Device:C
- removed D?: LED, LED_THT:LED_D5.0mm, symbol Device:LED
- removed D?: 2.7v, Diode_THT:D_DO-15_P12.70mm_Horizontal, symbol Device:D_Zener
- removed J?: DEBUG, Connector_PinHeader_2.54mm:PinHeader_2x07_P2.54mm_Vertical, symbol Connector_Generic:Conn_02x07_Odd_Even
- removed Q? (x2): choose me, Package_TO_SOT_THT:TO-220-3_Vertical, symbol Transistor_FET:IRF540N
- removed Q? (x2): AP2301GN, Package_TO_SOT_SMD:SOT-23, symbol Transistor_FET:TP0610T
- removed Q? (x2): IRF540N, Package_TO_SOT_THT:TO-220-3_Vertical, symbol Transistor_FET:IRF540N
- removed R? (x4): 4.7k, Resistor_SMD:R_0805_2012Metric_Pad1.15x1.40mm_HandSolder, symbol Device:R
- removed R? (x2): 22k, Potentiometer_THT:Potentiometer_Bourns_3296Y_Vertical, symbol Device:R_Potentiometer_Trim
- removed R? (x7): 10k, symbol Device:R
- removed R?: 47k, symbol Device:R
- removed R?: 1.2k, Resistor_THT:R_Axial_DIN0309_L9.0mm_D3.2mm_P12.70mm_Horizontal, symbol Device:R
- removed R?: 150k, Resistor_SMD:R_0805_2012Metric_Pad1.15x1.40mm_HandSolder, symbol Device:R
- removed R? (x2): 10k, Resistor_SMD:R_0805_2012Metric_Pad1.15x1.40mm_HandSolder, symbol Device:R
- removed R?: LDR03, OptoDevice:R_LDR_10x8.5mm_P7.6mm_Vertical, symbol Sensor_Optical:LDR03
- removed SW? (x2): BUTTON, Connector_PinHeader_2.54mm:PinHeader_1x02_P2.54mm_Vertical, symbol Switch:SW_Push
- removed SW?: SW_Push_DPDT, symbol Switch:SW_Push_DPDT
- removed TP?: TestPoint, TestPoint:TestPoint_THTPad_D2.0mm_Drill1.0mm, symbol Connector:TestPoint_Alt
- removed U? (x5): LM324, Package_SO:SOIC-14_3.9x8.7mm_P1.27mm, symbol Amplifier_Operational:LM324
- removed U?: LMC7660, Package_SO:SOIC-8_3.9x4.9mm_P1.27mm, symbol Regulator_SwitchedCapacitor:LMC7660
- removed U?: ESP-12E, RF_Module:ESP-12E, symbol RF_Module:ESP-12E
- added C? (x2): 10µ, Capacitor_SMD:C_1206_3216Metric_Pad1.33x1.80mm_HandSolder, symbol Device:C_Polarized
- added C? (x2): 100n, Capacitor_SMD:C_0805_2012Metric_Pad1.18x1.45mm_HandSolder, symbol Device:C
- added C?: x, symbol Device:C
- added C?: 10p, Capacitor_SMD:C_0805_2012Metric_Pad1.18x1.45mm_HandSolder, symbol Device:C
- added JP?: pwm_or_analog, symbol Jumper:Jumper_2_Bridged
- added JP?: mosfet_or_direct, symbol Jumper:Jumper_3_Bridged12
- added JP?: hard_onoff, symbol Jumper:Jumper_2_Bridged
- added Q?: choose me, Package_TO_SOT_THT:TO-220-3_Vertical, symbol Transistor_FET:IRF540N
- added Q?: AP2301GN, Package_TO_SOT_SMD:SOT-23, symbol Transistor_FET:TP0610T
- added Q?: IRF540N, Package_TO_SOT_THT:TO-220-3_Vertical, symbol Transistor_FET:IRF540N
- added R?: 47k, symbol Device:R
- added R? (x3): 22k, symbol Device:R
- added R? (x2): 100, symbol Device:R
- added R?: 2.2k, symbol Device:R
- added R? (x5): 10k, symbol Device:R
- added R?: 10k, Potentiometer_THT:Potentiometer_Bourns_3296Y_Vertical, symbol Device:R_Potentiometer_Trim
- added R?: 22k, Potentiometer_THT:Potentiometer_Bourns_3296Y_Vertical, symbol Device:R_Potentiometer_Trim
- added TP?: TestPoint, TestPoint:TestPoint_THTPad_D2.0mm_Drill1.0mm, symbol Connector:TestPoint_Alt
- added U? (x3): LM324, Package_SO:SOIC-14_3.9x8.7mm_P1.27mm, symbol Amplifier_Operational:LM324
- added U?: TL431, Package_TO_SOT_SMD:SOT-363_SC-70-6, symbol Reference_Voltage:TL431DCK
- added U?: LMC7660, Package_SO:SOIC-8_3.9x4.9mm_P1.27mm, symbol Regulator_SwitchedCapacitor:LMC7660
Connections:
- net VDD is gone; now on net VCC: C?.1, U?.4 (V+)
- net +3V3: now also C?.1, C?.1, R?.1, U?.8 (V+)
- net -VSW: now also C?.1, C?.2, TP?.1, U?.5 (VOUT)
- net GND: now also C?.1, C?.2, C?.2, JP?.2 (B), Q?.3 (S), Q?.3 (S), R?.1, R?.2, R?.2, R?.2, R?.2, U?.3 (GND), U?.6 (A), U?.6 (LV)
- net OUT1: now also JP?.1 (A), Q?.2 (D)
- net PWM1: now also U?.2 (-)
- net TRIANGLE: now also JP?.2 (B)
- net VCC: now also R?.1
- net VREF: now also Q?.3 (D), R?.1, R?.1, R?.1, R?.2, U?.1
- net at U?.3 (+): now also R?.1, R?.2
- net at D?.2 (A), U?.1: now also R?.1
- net at U?.2 (-): now also R?.1, R?.2
- net at C?.1, U?.2 (-): now also R?.1, R?.2
- new net: C?.1, U?.2 (CAP+)
- new net: C?.2, U?.4 (CAP-)
- new net: JP?.1 (A), R?.1, U?.2 (-)
- new net: JP?.2 (C), R?.2, U?.1
- new net: C?.2, R?.2, U?.3 (+)
- new net: R?.2, R?.3, U?.2 (-)
- new net: R?.2, U?.1 (K), U?.3 (+), U?.3 (REF)
- new net: JP?.3 (B), Q?.1 (G), R?.1
- new net: C?.2, U?.7 (OSC)
- new net: C?.1, JP?.1 (A)
- new net: Q?.1 (G), Q?.1 (G), U?.1
- new net: Q?.2 (D), Q?.2 (S), R?.1
- new net: R?.2, R?.3
- new net: R?.1, R?.2, U?.3 (+)
- no-connect marks 9 -> 0
Other:
- note added: "adjust freq"
- note added: "adjust so that there is no pwm at max duty"
- note added: "adjust so that there is no pwm at min duty"
- moved on the sheet: C?, R?, U?A
