File: boards/high_power_lamp/fast_pwm_controller/pwm_stage.kicad_sch (KiCad schematic)
At the start: 8 parts, among them Q4 BUK7516-55A,127, U1 4050, U2 TLC3704

Commit message: finalise board
Parts:
- added TP3, TP4: TestPoint, TestPoint:TestPoint_THTPad_D2.0mm_Drill1.0mm, symbol Connector:TestPoint
- renumbered Q4 to Q1, R26 to R13
Connections:
- net at R13.2, U2.14: now also TP4.1
- net at C8.2, R12.1, U2.9 (+): now also TP3.1
Other:
- moved on the sheet: R13
Changed lines of the file:
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@@
   (junction (at 82.55 81.28) (diameter 0) (color 0 0 0 0)
   )
+  (junction (at 167.64 83.82) (diameter 0) (color 0 0 0 0)
+  )
   (junction (at 105.41 81.28) (diameter 0) (color 0 0 0 0)
   )
+  (junction (at 143.51 81.28) (diameter 0) (color 0 0 0 0)
+  )
   (junction (at 119.38 81.28) (diameter 0) (color 0 0 0 0)
   )
@@
     (stroke (width 0) (type default))
   )
+  (wire (pts (xy 177.8 83.82) (xy 181.61 83.82))
+    (stroke (width 0) (type default))
+  )
+  (wire (pts (xy 143.51 81.28) (xy 149.86 81.28))
+    (stroke (width 0) (type default))
+  )
   (wire (pts (xy 189.23 78.74) (xy 189.23 71.12))
     (stroke (width 0) (type default))
@@
     (stroke (width 0) (type default))
   )
-  (wire (pts (xy 165.1 83.82) (xy 168.91 83.82))
+  (wire (pts (xy 165.1 83.82) (xy 167.64 83.82))
     (stroke (width 0) (type default))
   )
@@
     (stroke (width 0) (type default))
   )
+  (wire (pts (xy 167.64 83.82) (xy 170.18 83.82))
+    (stroke (width 0) (type default))
+  )
   (wire (pts (xy 146.05 86.36) (xy 149.86 86.36))
     (stroke (width 0) (type default))
@@
     (stroke (width 0) (type default))
   )
-  (wire (pts (xy 119.38 81.28) (xy 149.86 81.28))
-    (stroke (width 0) (type default))
-  )
-  (wire (pts (xy 176.53 83.82) (xy 181.61 83.82))
+  (wire (pts (xy 119.38 81.28) (xy 143.51 81.28))
     (stroke (width 0) (type default))
   )
@@
     )
   )
-  (symbol (lib_id "Device:R") (at 172.72 83.82 270) (unit 1)
-    (in_bom yes) (on_board yes) (dnp no)
-    (property "Reference" "R26" (at 172.72 86.36 90)
-      (effects (font (size 1.27 1.27)))
-    )
-    (property "Value" "2.2Ω" (at 172.72 88.9 90)
-      (effects (font (size 1.27 1.27)))
-    )
-    (property "Footprint" "Resistor_SMD:R_0805_2012Metric" (at 172.72 82.042 90)
-      (effects (font (size 1.27 1.27)) hide)
-    )
-    (property "Datasheet" "~" (at 172.72 83.82 0)
-      (effects (font (size 1.27 1.27)) hide)
-    )
-    (pin "1")
-    (pin "2")
-    (instances
-      (project "fast_pwm_controller"
-        (path "/ebb02bb0-15d4-41b5-b7b0-053d51d38d86/1dc02105-34f4-4dcd-909a-a43f3cf6326e"
+  (symbol (lib_id "Device:R") (at 173.99 83.82 270) (unit 1)
+    (in_bom yes) (on_board yes) (dnp no)
+    (property "Reference" "R13" (at 173.99 86.36 90)
+      (effects (font (size 1.27 1.27)))
+    )
+    (property "Value" "2.2Ω" (at 173.99 88.9 90)
+      (effects (font (size 1.27 1.27)))
+    )
+    (property "Footprint" "Resistor_SMD:R_0805_2012Metric" (at 173.99 82.042 90)
+      (effects (font (size 1.27 1.27)) hide)
+    )
+    (property "Datasheet" "~" (at 173.99 83.82 0)
+      (effects (font (size 1.27 1.27)) hide)
+    )
+    (pin "1")
+    (pin "2")
+    (instances
+      (project "fast_pwm_controller"
+        (path "/ebb02bb0-15d4-41b5-b7b0-053d51d38d86/1dc02105-34f4-4dcd-909a-a43f3cf6326e"
+          (reference "R13") (unit 1)
+        )
+        (path "/ebb02bb0-15d4-41b5-b7b0-053d51d38d86/7bb7f3cd-bd16-48a2-9709-ee0db83f3451"
+          (reference "R20") (unit 1)
+        )
+        (path "/ebb02bb0-15d4-41b5-b7b0-053d51d38d86/abcbc788-820f-4167-8f5b-0037e0acabb5"
+          (reference "R23") (unit 1)
+        )
+        (path "/ebb02bb0-15d4-41b5-b7b0-053d51d38d86/7c02a172-be14-404a-b556-b25540aed647"
           (reference "R26") (unit 1)
-        )
-        (path "/ebb02bb0-15d4-41b5-b7b0-053d51d38d86/7bb7f3cd-bd16-48a2-9709-ee0db83f3451"
-          (reference "R23") (unit 1)
-        )
-        (path "/ebb02bb0-15d4-41b5-b7b0-053d51d38d86/abcbc788-820f-4167-8f5b-0037e0acabb5"
-          (reference "R13") (unit 1)
-        )
-        (path "/ebb02bb0-15d4-41b5-b7b0-053d51d38d86/7c02a172-be14-404a-b556-b25540aed647"
-          (reference "R20") (unit 1)
         )
       )
@@
         (path "/ebb02bb0-15d4-41b5-b7b0-053d51d38d86/7c02a172-be14-404a-b556-b25540aed647"
           (reference "R24") (unit 1)
+        )
+      )
+    )
+  )
+  (symbol (lib_id "Connector:TestPoint") (at 143.51 81.28 0) (unit 1)
+    (in_bom yes) (on_board yes) (dnp no)
+    (property "Reference" "TP3" (at 142.24 76.2 0)
+      (effects (font (size 1.27 1.27)) (justify left))
+    )
+    (property "Value" "TestPoint" (at 146.05 79.248 0)
+      (effects (font (size 1.27 1.27)) (justify left) hide)
+    )
+    (property "Footprint" "TestPoint:TestPoint_THTPad_D2.0mm_Drill1.0mm" (at 148.59 81.28 0)
+      (effects (font (size 1.27 1.27)) hide)
+    )
+    (property "Datasheet" "~" (at 148.59 81.28 0)
+      (effects (font (size 1.27 1.27)) hide)
+    )
+    (pin "1")
+    (instances
+      (project "fast_pwm_controller"
+        (path "/ebb02bb0-15d4-41b5-b7b0-053d51d38d86/1dc02105-34f4-4dcd-909a-a43f3cf6326e"
+          (reference "TP3") (unit 1)
+        )
+        (path "/ebb02bb0-15d4-41b5-b7b0-053d51d38d86/7bb7f3cd-bd16-48a2-9709-ee0db83f3451"
+          (reference "TP5") (unit 1)
+        )
+        (path "/ebb02bb0-15d4-41b5-b7b0-053d51d38d86/abcbc788-820f-4167-8f5b-0037e0acabb5"
+          (reference "TP7") (unit 1)
+        )
+        (path "/ebb02bb0-15d4-41b5-b7b0-053d51d38d86/7c02a172-be14-404a-b556-b25540aed647"
+          (reference "TP9") (unit 1)
+        )
+      )
+    )
+  )
+  (symbol (lib_id "Connector:TestPoint") (at 167.64 83.82 0) (unit 1)
+    (in_bom yes) (on_board yes) (dnp no)
+    (property "Reference" "TP4" (at 166.37 78.74 0)
+      (effects (font (size 1.27 1.27)) (justify left))
+    )
+    (property "Value" "TestPoint" (at 170.18 81.788 0)
+      (effects (font (size 1.27 1.27)) (justify left) hide)
+    )
+    (property "Footprint" "TestPoint:TestPoint_THTPad_D2.0mm_Drill1.0mm" (at 172.72 83.82 0)
+      (effects (font (size 1.27 1.27)) hide)
+    )
+    (property "Datasheet" "~" (at 172.72 83.82 0)
+      (effects (font (size 1.27 1.27)) hide)
+    )
+    (pin "1")
+    (instances
+      (project "fast_pwm_controller"
+        (path "/ebb02bb0-15d4-41b5-b7b0-053d51d38d86/1dc02105-34f4-4dcd-909a-a43f3cf6326e"
+          (reference "TP4") (unit 1)
+        )
+        (path "/ebb02bb0-15d4-41b5-b7b0-053d51d38d86/7bb7f3cd-bd16-48a2-9709-ee0db83f3451"
+          (reference "TP6") (unit 1)
+        )
+        (path "/ebb02bb0-15d4-41b5-b7b0-053d51d38d86/abcbc788-820f-4167-8f5b-0037e0acabb5"
+          (reference "TP8") (unit 1)
+        )
+        (path "/ebb02bb0-15d4-41b5-b7b0-053d51d38d86/7c02a172-be14-404a-b556-b25540aed647"
+          (reference "TP10") (unit 1)
         )
       )
@@
   (symbol (lib_id "Device:Q_NMOS_GDS") (at 186.69 83.82 0) (unit 1)
     (in_bom yes) (on_board yes) (dnp no) (fields_autoplaced)
-    (property "Reference" "Q4" (at 193.04 83.82 0)
+    (property "Reference" "Q1" (at 193.04 83.82 0)
       (effects (font (size 1.27 1.27)) (justify left))
     )
@@
       (project "fast_pwm_controller"
         (path "/ebb02bb0-15d4-41b5-b7b0-053d51d38d86/1dc02105-34f4-4dcd-909a-a43f3cf6326e"
+          (reference "Q1") (unit 1)
+        )
+        (path "/ebb02bb0-15d4-41b5-b7b0-053d51d38d86/7bb7f3cd-bd16-48a2-9709-ee0db83f3451"
+          (reference "Q2") (unit 1)
+        )
+        (path "/ebb02bb0-15d4-41b5-b7b0-053d51d38d86/abcbc788-820f-4167-8f5b-0037e0acabb5"
+          (reference "Q3") (unit 1)
+        )
+        (path "/ebb02bb0-15d4-41b5-b7b0-053d51d38d86/7c02a172-be14-404a-b556-b25540aed647"
           (reference "Q4") (unit 1)
         )
-        (path "/ebb02bb0-15d4-41b5-b7b0-053d51d38d86/7bb7f3cd-bd16-48a2-9709-ee0db83f3451"
-          (reference "Q3") (unit 1)
-        )
-        (path "/ebb02bb0-15d4-41b5-b7b0-053d51d38d86/abcbc788-820f-4167-8f5b-0037e0acabb5"
-          (reference "Q1") (unit 1)
-        )
-        (path "/ebb02bb0-15d4-41b5-b7b0-053d51d38d86/7c02a172-be14-404a-b556-b25540aed647"
-          (reference "Q2") (unit 1)
-        )
-      )
+      )

Commit message: finalise pcb
Parts:
- renumbered C8 to C17, JP1 to JP4, Q1 to Q2, R13 to R20, R11 to R21, R12 to R22, TP3 to TP7
Connections:
- net IN: now also U1.9; no longer U1.7
- net at JP4.2 (B), R22.2: now also U1.10; no longer U1.6
Changed lines of the file:
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@@
   (symbol (lib_id "Device:R") (at 111.76 81.28 270) (unit 1)
     (in_bom yes) (on_board yes) (dnp no)
-    (property "Reference" "R12" (at 111.76 83.82 90)
+    (property "Reference" "R22" (at 111.76 83.82 90)
       (effects (font (size 1.27 1.27)))
     )
@@
       (project "fast_pwm_controller"
         (path "/ebb02bb0-15d4-41b5-b7b0-053d51d38d86/1dc02105-34f4-4dcd-909a-a43f3cf6326e"
+          (reference "R22") (unit 1)
+        )
+        (path "/ebb02bb0-15d4-41b5-b7b0-053d51d38d86/7bb7f3cd-bd16-48a2-9709-ee0db83f3451"
           (reference "R12") (unit 1)
         )
-        (path "/ebb02bb0-15d4-41b5-b7b0-053d51d38d86/7bb7f3cd-bd16-48a2-9709-ee0db83f3451"
+        (path "/ebb02bb0-15d4-41b5-b7b0-053d51d38d86/abcbc788-820f-4167-8f5b-0037e0acabb5"
           (reference "R19") (unit 1)
-        )
-        (path "/ebb02bb0-15d4-41b5-b7b0-053d51d38d86/abcbc788-820f-4167-8f5b-0037e0acabb5"
-          (reference "R22") (unit 1)
         )
         (path "/ebb02bb0-15d4-41b5-b7b0-053d51d38d86/7c02a172-be14-404a-b556-b25540aed647"
@@
   (symbol (lib_id "Device:R") (at 173.99 83.82 270) (unit 1)
     (in_bom yes) (on_board yes) (dnp no)
-    (property "Reference" "R13" (at 173.99 86.36 90)
+    (property "Reference" "R20" (at 173.99 86.36 90)
       (effects (font (size 1.27 1.27)))
     )
@@
       (project "fast_pwm_controller"
         (path "/ebb02bb0-15d4-41b5-b7b0-053d51d38d86/1dc02105-34f4-4dcd-909a-a43f3cf6326e"
+          (reference "R20") (unit 1)
+        )
+        (path "/ebb02bb0-15d4-41b5-b7b0-053d51d38d86/7bb7f3cd-bd16-48a2-9709-ee0db83f3451"
+          (reference "R26") (unit 1)
+        )
+        (path "/ebb02bb0-15d4-41b5-b7b0-053d51d38d86/abcbc788-820f-4167-8f5b-0037e0acabb5"
           (reference "R13") (unit 1)
         )
-        (path "/ebb02bb0-15d4-41b5-b7b0-053d51d38d86/7bb7f3cd-bd16-48a2-9709-ee0db83f3451"
-          (reference "R20") (unit 1)
-        )
-        (path "/ebb02bb0-15d4-41b5-b7b0-053d51d38d86/abcbc788-820f-4167-8f5b-0037e0acabb5"
+        (path "/ebb02bb0-15d4-41b5-b7b0-053d51d38d86/7c02a172-be14-404a-b556-b25540aed647"
           (reference "R23") (unit 1)
         )
-        (path "/ebb02bb0-15d4-41b5-b7b0-053d51d38d86/7c02a172-be14-404a-b556-b25540aed647"
-          (reference "R26") (unit 1)
-        )
       )
     )
@@
   (symbol (lib_id "Jumper:SolderJumper_2_Open") (at 93.98 66.04 0) (unit 1)
     (in_bom yes) (on_board yes) (dnp no)
-    (property "Reference" "JP1" (at 93.98 63.5 0)
+    (property "Reference" "JP4" (at 93.98 63.5 0)
       (effects (font (size 1.27 1.27)))
     )
@@
       (project "fast_pwm_controller"
         (path "/ebb02bb0-15d4-41b5-b7b0-053d51d38d86/1dc02105-34f4-4dcd-909a-a43f3cf6326e"
+          (reference "JP4") (unit 1)
+        )
+        (path "/ebb02bb0-15d4-41b5-b7b0-053d51d38d86/7bb7f3cd-bd16-48a2-9709-ee0db83f3451"
           (reference "JP1") (unit 1)
         )
-        (path "/ebb02bb0-15d4-41b5-b7b0-053d51d38d86/7bb7f3cd-bd16-48a2-9709-ee0db83f3451"
+        (path "/ebb02bb0-15d4-41b5-b7b0-053d51d38d86/abcbc788-820f-4167-8f5b-0037e0acabb5"
           (reference "JP3") (unit 1)
-        )
-        (path "/ebb02bb0-15d4-41b5-b7b0-053d51d38d86/abcbc788-820f-4167-8f5b-0037e0acabb5"
-          (reference "JP4") (unit 1)
         )
         (path "/ebb02bb0-15d4-41b5-b7b0-053d51d38d86/7c02a172-be14-404a-b556-b25540aed647"
@@
   (symbol (lib_id "Device:C") (at 119.38 88.9 180) (unit 1)
     (in_bom yes) (on_board yes) (dnp no)
-    (property "Reference" "C8" (at 123.19 86.36 0)
+    (property "Reference" "C17" (at 123.19 86.36 0)
       (effects (font (size 1.27 1.27)) (justify right))
     )
@@
       (project "fast_pwm_controller"
         (path "/ebb02bb0-15d4-41b5-b7b0-053d51d38d86/1dc02105-34f4-4dcd-909a-a43f3cf6326e"
+          (reference "C17") (unit 1)
+        )
+        (path "/ebb02bb0-15d4-41b5-b7b0-053d51d38d86/7bb7f3cd-bd16-48a2-9709-ee0db83f3451"
           (reference "C8") (unit 1)
         )
-        (path "/ebb02bb0-15d4-41b5-b7b0-053d51d38d86/7bb7f3cd-bd16-48a2-9709-ee0db83f3451"
+        (path "/ebb02bb0-15d4-41b5-b7b0-053d51d38d86/abcbc788-820f-4167-8f5b-0037e0acabb5"
           (reference "C16") (unit 1)
         )
-        (path "/ebb02bb0-15d4-41b5-b7b0-053d51d38d86/abcbc788-820f-4167-8f5b-0037e0acabb5"
-          (reference "C17") (unit 1)
-        )
         (path "/ebb02bb0-15d4-41b5-b7b0-053d51d38d86/7c02a172-be14-404a-b556-b25540aed647"
           (reference "C18") (unit 1)
@@
   (symbol (lib_id "Device:R") (at 82.55 88.9 0) (unit 1)
     (in_bom yes) (on_board yes) (dnp no)
-    (property "Reference" "R11" (at 85.09 87.63 0)
+    (property "Reference" "R21" (at 85.09 87.63 0)
       (effects (font (size 1.27 1.27)) (justify left))
     )
@@
       (project "fast_pwm_controller"
         (path "/ebb02bb0-15d4-41b5-b7b0-053d51d38d86/1dc02105-34f4-4dcd-909a-a43f3cf6326e"
+          (reference "R21") (unit 1)
+        )
+        (path "/ebb02bb0-15d4-41b5-b7b0-053d51d38d86/7bb7f3cd-bd16-48a2-9709-ee0db83f3451"
           (reference "R11") (unit 1)
         )
-        (path "/ebb02bb0-15d4-41b5-b7b0-053d51d38d86/7bb7f3cd-bd16-48a2-9709-ee0db83f3451"
+        (path "/ebb02bb0-15d4-41b5-b7b0-053d51d38d86/abcbc788-820f-4167-8f5b-0037e0acabb5"
           (reference "R18") (unit 1)
         )
-        (path "/ebb02bb0-15d4-41b5-b7b0-053d51d38d86/abcbc788-820f-4167-8f5b-0037e0acabb5"
-          (reference "R21") (unit 1)
-        )
         (path "/ebb02bb0-15d4-41b5-b7b0-053d51d38d86/7c02a172-be14-404a-b556-b25540aed647"
           (reference "R24") (unit 1)
@@
   (symbol (lib_id "Connector:TestPoint") (at 143.51 81.28 0) (unit 1)
     (in_bom yes) (on_board yes) (dnp no)
-    (property "Reference" "TP3" (at 142.24 76.2 0)
+    (property "Reference" "TP7" (at 142.24 76.2 0)
       (effects (font (size 1.27 1.27)) (justify left))
     )
@@
       (project "fast_pwm_controller"
         (path "/ebb02bb0-15d4-41b5-b7b0-053d51d38d86/1dc02105-34f4-4dcd-909a-a43f3cf6326e"
+          (reference "TP7") (unit 1)
+        )
+        (path "/ebb02bb0-15d4-41b5-b7b0-053d51d38d86/7bb7f3cd-bd16-48a2-9709-ee0db83f3451"
           (reference "TP3") (unit 1)
         )
-        (path "/ebb02bb0-15d4-41b5-b7b0-053d51d38d86/7bb7f3cd-bd16-48a2-9709-ee0db83f3451"
+        (path "/ebb02bb0-15d4-41b5-b7b0-053d51d38d86/abcbc788-820f-4167-8f5b-0037e0acabb5"
           (reference "TP5") (unit 1)
-        )
-        (path "/ebb02bb0-15d4-41b5-b7b0-053d51d38d86/abcbc788-820f-4167-8f5b-0037e0acabb5"
-          (reference "TP7") (unit 1)
         )
         (path "/ebb02bb0-15d4-41b5-b7b0-053d51d38d86/7c02a172-be14-404a-b556-b25540aed647"
@@
     )
   )
-  (symbol (lib_id "4xxx:4050") (at 95.25 81.28 0) (unit 3)
+  (symbol (lib_id "4xxx:4050") (at 95.25 81.28 0) (unit 4)
     (in_bom yes) (on_board yes) (dnp no) (fields_autoplaced)
     (property "Reference" "U1" (at 95.25 72.39 0)
@@
       (project "fast_pwm_controller"
         (path "/ebb02bb0-15d4-41b5-b7b0-053d51d38d86/1dc02105-34f4-4dcd-909a-a43f3cf6326e"
+          (reference "U1") (unit 4)
+        )
+        (path "/ebb02bb0-15d4-41b5-b7b0-053d51d38d86/7bb7f3cd-bd16-48a2-9709-ee0db83f3451"
           (reference "U1") (unit 3)
         )
-        (path "/ebb02bb0-15d4-41b5-b7b0-053d51d38d86/7bb7f3cd-bd16-48a2-9709-ee0db83f3451"
+        (path "/ebb02bb0-15d4-41b5-b7b0-053d51d38d86/abcbc788-820f-4167-8f5b-0037e0acabb5"
           (reference "U1") (unit 1)
-        )
-        (path "/ebb02bb0-15d4-41b5-b7b0-053d51d38d86/abcbc788-820f-4167-8f5b-0037e0acabb5"
-          (reference "U1") (unit 4)
         )
         (path "/ebb02bb0-15d4-41b5-b7b0-053d51d38d86/7c02a172-be14-404a-b556-b25540aed647"
@@
   (symbol (lib_id "Device:Q_NMOS_GDS") (at 186.69 83.82 0) (unit 1)
     (in_bom yes) (on_board yes) (dnp no) (fields_autoplaced)
-    (property "Reference" "Q1" (at 193.04 83.82 0)
+    (property "Reference" "Q2" (at 193.04 83.82 0)
       (effects (font (size 1.27 1.27)) (justify left))
     )
@@
       (project "fast_pwm_controller"
         (path "/ebb02bb0-15d4-41b5-b7b0-053d51d38d86/1dc02105-34f4-4dcd-909a-a43f3cf6326e"
+          (reference "Q2") (unit 1)
+        )
+        (path "/ebb02bb0-15d4-41b5-b7b0-053d51d38d86/7bb7f3cd-bd16-48a2-9709-ee0db83f3451"
+          (reference "Q4") (unit 1)
+        )
+        (path "/ebb02bb0-15d4-41b5-b7b0-053d51d38d86/abcbc788-820f-4167-8f5b-0037e0acabb5"
           (reference "Q1") (unit 1)
         )
-        (path "/ebb02bb0-15d4-41b5-b7b0-053d51d38d86/7bb7f3cd-bd16-48a2-9709-ee0db83f3451"
-          (reference "Q2") (unit 1)
-        )
-        (path "/ebb02bb0-15d4-41b5-b7b0-053d51d38d86/abcbc788-820f-4167-8f5b-0037e0acabb5"
+        (path "/ebb02bb0-15d4-41b5-b7b0-053d51d38d86/7c02a172-be14-404a-b556-b25540aed647"
           (reference "Q3") (unit 1)
         )
-        (path "/ebb02bb0-15d4-41b5-b7b0-053d51d38d86/7c02a172-be14-404a-b556-b25540aed647"
-          (reference "Q4") (unit 1)
-        )
-      )
+      )
