File: boards/high_power_lamp/fast_pwm_controller/fast_pwm_controller.kicad_sch (KiCad schematic)
At the start: 35 parts, among them J1 Screw_Terminal_01x01, J10 Screw_Terminal_01x01, J11 Screw_Terminal_01x01, J12 Screw_Terminal_01x01, J13 Screw_Terminal_01x01, J14 Screw_Terminal_01x01, J15 Screw_Terminal_01x01, J16 Screw_Terminal_01x01, J17 Screw_Terminal_01x01, J18 Screw_Terminal_01x01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

Commit message: final touches to the fast pwm controller
Parts:
- J1: Purpose VPP IN -> VPP-IN
Changed lines of the file:
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@@
       (effects (font (size 1.27 1.27)) hide)
     )
-    (property "Purpose" "VPP IN" (at 73.66 36.83 0)
+    (property "Purpose" "VPP-IN" (at 73.66 36.83 0)
       (effects (font (size 1.27 1.27)) (justify left))
     )
